File: Video Gen.kicad_sch (KiCad schematic)
At the start: 35 parts, among them J18 Aux Video, K14 VIDEO OUT, Q3 2N3904

Commit message: Add files via upload
Connections:
- net GND: now also A8.13 (I1c)
- net LD7: no longer A8.13 (I1c)
Changed lines of the file:
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@@
     (stroke (width 0) (type default))
   )
+  (wire (pts (xy 248.92 165.1) (xy 248.92 167.64))
+    (stroke (width 0) (type default))
+  )
   (wire (pts (xy 302.768 205.74) (xy 303.784 205.74))
     (stroke (width 0) (type default))
@@
     (stroke (width 0) (type default))
   )
-  (wire (pts (xy 265.43 165.1) (xy 267.97 165.1))
+  (wire (pts (xy 248.92 165.1) (xy 267.97 165.1))
     (stroke (width 0) (type default))
   )
@@
     )
   )
-  (global_label "LD7" (shape input) (at 265.43 165.1 180)
-    (effects (font (size 1.27 1.27)) (justify right))
-    (property "Intersheetrefs" "${INTERSHEET_REFS}" (at 265.43 165.1 0)
-      (effects (font (size 1.27 1.27)) hide)
-    )
-  )
   (global_label "LD194" (shape input) (at 377.19 161.036 0)
     (effects (font (size 1.27 1.27)) (justify left))
@@
         )
       )
+    )
+  )
+  (symbol (lib_id "power:GND") (at 248.92 167.64 0) (unit 1)
+    (in_bom yes) (on_board yes) (dnp no)
+    (property "Reference" "#PWR03" (at 248.92 173.99 0)
+      (effects (font (size 1.27 1.27)) hide)
+    )
+    (property "Value" "GND" (at 246.634 170.434 0)
+      (effects (font (size 1.27 1.27)))
+    )
+    (property "Footprint" "" (at 248.92 167.64 0)
+      (effects (font (size 1.27 1.27)) hide)
+    )
+    (property "Datasheet" "" (at 248.92 167.64 0)
+      (effects (font (size 1.27 1.27)) hide)
+    )
+    (pin "1")
+    (instances
+      (project "AppleII"
+        (path "/f1f08369-4db3-46f7-9b89-a5d3cfbed55a/00000000-0000-0000-0000-0000632bf564"
+          (reference "#PWR03") (unit 1)
+        )
+      )

Commit message: Add files via upload
Other:
- note added: "Mixer"
- note added: "Sync Generator"
- note added: "Video Generator"
- moved on the sheet: A10, A3, A5, A8, A9, B10A, B11B, B11C, B11D, B12A, B12B, B13A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

Commit message: Add files via upload
Parts:
- removed A10: 74LS194, Package_DIP:DIP-16_W7.62mm_Socket, symbol AppleII+:74LS194
- added A10: 74LS194, Apple:DIP-16_W7.62mm, symbol 74xx:74LS194
Connections:
- net +5V: now also A10.16 (VCC)
- net 14M: now also A10.11 (Cp)
- net A3-2: now also A10.6 (P3)
- net A8-3-A9-B9: no longer A8.3 (I1a), A9.13 (I6), B9.15 (Q0)
- net C14-6: now also A10.5 (P2)
- net GND: now also A10.8 (GND)
- net LD194: now also A10.10 (S1), A10.9 (S0)
- net SOFT5: now also A10.1 (Mr), A10.2 (Dsr), A10.7 (Dsl)
- net at A9.10 (S1): now also A10.15 (Q0)
- net at A9.11 (S0): now also A10.14 (Q1)
- net at A9.7 (~{E}): now also A10.13 (Q2)
- net A8-7: now reaches A8.7 (Zb)
- net A8-7: now also A10.3 (P0)
- net A8-12: now reaches A8.12 (Zc)
- net A8-12: now also A10.4 (P1)
- net A3-1: no longer names the net of A3.1 (Ds), B2.12
- net A3-1: now also A10.12 (Q3)
- net B9-13: no longer names the net of A9.12 (I7), B9.13 (Q2)
- new net: A8.3 (I1a), A9.13 (I6), B9.15 (Q0)
Other:
- note added: "Composite Video Output"
- note added: "Data Selector"
- note added: "Flashing"
- note added: "Graphics Shift Register"
- note added: "Inverse Video"
- note added: "LD6"
- note added: "LD7"
- note added: "Note: See Data Latch."
- note added: "Shift Register"
- note added: "Shift Register Configuration"
- note removed: "Note: See RAM circuit."
- moved on the sheet: A8, B11B, B12B, B13D, Cap13, Cap14, J18, K14, R10, R11

Commit message: Add files via upload
Other:
- moved on the sheet: B12B, Cap13, Cap14, R10

Commit message: Add files via upload
Parts:
- added unit 5 of B13
- added unit 3 of C13
- added unit 5 of C14
Connections:
- net +5V: now also B13.14 (VCC), C13.14 (VCC), C14.14 (VCC)
- net GND: now also B13.7 (GND), C13.7 (GND), C14.7 (GND)
- net A9-9 renamed B11-5
Other:
- note added: "H[0..5]"
- note added: "V[0..5]"

Commit message: Add files via upload
Parts:
- added unit 5 of A2
Connections:
- net +5V: now also A2.14 (VCC)
- net GND: now also A2.7 (GND)
Changed lines of the file:
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@@
   (junction (at 315.468 80.01) (diameter 0) (color 0 0 0 0)
   )
+  (junction (at 110.49 397.51) (diameter 0) (color 0 0 0 0)
+  )
   (junction (at 457.2 236.22) (diameter 0) (color 0 0 0 0)
   )
@@
   (junction (at 435.61 182.88) (diameter 0) (color 0 0 0 0)
   )
+  (junction (at 95.25 367.03) (diameter 0) (color 0 0 0 0)
+  )
   (junction (at 315.468 56.642) (diameter 0) (color 0 0 0 0)
   )
@@
     (stroke (width 0) (type default))
   )
-  (wire (pts (xy 110.49 364.49) (xy 110.49 367.03))
-    (stroke (width 0) (type default))
-  )
   (wire (pts (xy 297.18 91.44) (xy 297.18 114.3))
     (stroke (width 0) (type default))
@@
     (stroke (width 0) (type default))
   )
+  (wire (pts (xy 95.25 394.97) (xy 95.25 397.51))
+    (stroke (width 0) (type default))
+  )
   (wire (pts (xy 373.38 307.34) (xy 400.05 307.34))
     (stroke (width 0) (type default))
@@
     (stroke (width 0) (type default))
   )
+  (wire (pts (xy 95.25 369.57) (xy 95.25 367.03))
+    (stroke (width 0) (type default))
+  )
   (wire (pts (xy 396.24 322.58) (xy 400.05 322.58))
     (stroke (width 0) (type default))
@@
     (stroke (width 0) (type default))
   )
+  (wire (pts (xy 95.25 364.49) (xy 95.25 367.03))
+    (stroke (width 0) (type default))
+  )
   (wire (pts (xy 110.49 397.51) (xy 125.73 397.51))
     (stroke (width 0) (type default))
@@
     (stroke (width 0) (type default))
   )
+  (wire (pts (xy 95.25 397.51) (xy 110.49 397.51))
+    (stroke (width 0) (type default))
+  )
   (bus (pts (xy 25.4 31.75) (xy 55.88 31.75))
     (stroke (width 0) (type default))
@@
     (stroke (width 0) (type default))
   )
+  (wire (pts (xy 95.25 367.03) (xy 110.49 367.03))
+    (stroke (width 0) (type default))
+  )
   (wire (pts (xy 326.39 161.29) (xy 339.09 161.29))
     (stroke (width 0) (type default))
@@
     )
   )
-  (symbol (lib_id "power:+5V") (at 110.49 364.49 0) (unit 1)
+  (symbol (lib_id "power:+5V") (at 95.25 364.49 0) (unit 1)
     (in_bom yes) (on_board yes) (dnp no)
-    (property "Reference" "#PWR012" (at 110.49 368.3 0)
+    (property "Reference" "#PWR012" (at 95.25 368.3 0)
       (effects (font (size 1.27 1.27)) hide)
     )
-    (property "Value" "+5V" (at 113.03 362.712 0)
+    (property "Value" "+5V" (at 97.79 362.712 0)
       (effects (font (size 1.27 1.27)))
     )
-    (property "Footprint" "" (at 110.49 364.49 0)
+    (property "Footprint" "" (at 95.25 364.49 0)
       (effects (font (size 1.27 1.27)) hide)
     )
-    (property "Datasheet" "" (at 110.49 364.49 0)
+    (property "Datasheet" "" (at 95.25 364.49 0)
       (effects (font (size 1.27 1.27)) hide)
     )
@@
         )
       )
+    )
+  )
+  (symbol (lib_id "74xx:74LS00") (at 95.25 382.27 0) (unit 5)
+    (in_bom yes) (on_board yes) (dnp no)
+    (property "Reference" "A2" (at 96.52 373.38 0)
+      (effects (font (size 1.27 1.27)) (justify left))
+    )
+    (property "Value" "74LS00" (at 91.44 382.27 0)
+      (effects (font (size 1.27 1.27)) (justify left))
+    )
+    (property "Footprint" "" (at 95.25 382.27 0)
+      (effects (font (size 1.27 1.27)) hide)
+    )
+    (property "Datasheet" "http://www.ti.com/lit/gpn/sn74ls00" (at 95.25 382.27 0)
+      (effects (font (size 1.27 1.27)) hide)
+    )
+    (pin "3")
+    (pin "11")
+    (pin "7")
+    (pin "13")
+    (pin "12")
+    (pin "6")
+    (pin "9")
+    (pin "4")
+    (pin "14")
+    (pin "1")
+    (pin "10")
+    (pin "8")
+    (pin "5")
+    (pin "2")
+    (instances
+      (project "AppleII"
+        (path "/f1f08369-4db3-46f7-9b89-a5d3cfbed55a/00000000-0000-0000-0000-0000632bf564"
+          (reference "A2") (unit 5)
+        )
+      )

Commit message: Add files via upload
Connections:
- net A8-6 is gone; now on net GND: A8.6 (I1b)
Changed lines of the file:
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@@
   (junction (at 69.85 147.32) (diameter 0) (color 0 0 0 0)
+  )
+  (junction (at 303.53 213.36) (diameter 0) (color 0 0 0 0)
   )
   (junction (at 315.468 80.01) (diameter 0) (color 0 0 0 0)
@@
     (stroke (width 0) (type default))
   )
+  (wire (pts (xy 322.58 205.74) (xy 303.53 205.74))
+    (stroke (width 0) (type default))
+  )
   (wire (pts (xy 73.66 121.92) (xy 74.93 121.92))
     (stroke (width 0) (type default))
@@
     (stroke (width 0) (type default))
   )
-  (wire (pts (xy 320.04 205.74) (xy 322.58 205.74))
-    (stroke (width 0) (type default))
-  )
   (wire (pts (xy 322.58 195.58) (xy 322.58 185.42))
     (stroke (width 0) (type default))
@@
   )
   (wire (pts (xy 449.58 208.28) (xy 459.74 208.28))
+    (stroke (width 0) (type default))
+  )
+  (wire (pts (xy 303.53 205.74) (xy 303.53 213.36))
     (stroke (width 0) (type default))
   )
@@
     )
   )
-  (global_label "A8-6" (shape input) (at 320.04 205.74 180) (fields_autoplaced)
-    (effects (font (size 1.27 1.27)) (justify right))
-    (property "Intersheetrefs" "${INTERSHEET_REFS}" (at 312.629 205.74 0)
-      (effects (font (size 1.27 1.27)) (justify right) hide)
-    )
-  )

Commit message: Add files via upload
Connections:
- net SOFT5: no longer A2.8, A3.9 (Clr), B4.1 (Mr), B4.2 (Dsr)
- new net SOFT5a: A2.8, A3.9 (Clr), B4.1 (Mr), B4.2 (Dsr)
Changed lines of the file:
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@@
     )
   )
-  (global_label "SOFT5" (shape input) (at 379.73 163.83 180)
+  (global_label "SOFT5a" (shape input) (at 379.73 163.83 180)
     (effects (font (size 1.27 1.27)) (justify right))
     (property "Intersheetrefs" "${INTERSHEET_REFS}" (at 379.73 163.83 0)
@@
     )
   )
-  (global_label "SOFT5" (shape input) (at 399.034 270.51 180)
+  (global_label "SOFT5a" (shape input) (at 399.034 270.51 180)
     (effects (font (size 1.27 1.27)) (justify right))
     (property "Intersheetrefs" "${INTERSHEET_REFS}" (at 399.034 270.51 0)
@@
     )
   )
-  (global_label "SOFT5" (shape input) (at 399.034 250.19 180)
+  (global_label "SOFT5a" (shape input) (at 399.034 250.19 180)
     (effects (font (size 1.27 1.27)) (justify right))
     (property "Intersheetrefs" "${INTERSHEET_REFS}" (at 399.034 250.19 0)
@@
     )
   )
-  (global_label "SOFT5" (shape output) (at 54.61 372.11 0)
+  (global_label "SOFT5a" (shape output) (at 54.61 372.11 0)
     (effects (font (size 1.27 1.27)) (justify left))
     (property "Intersheetrefs" "${INTERSHEET_REFS}" (at 54.61 372.11 0)
