File: Video Gen.kicad_sch (KiCad schematic)
At the start: 35 parts, among them J18 Aux Video, K14 VIDEO OUT, Q3 2N3904

Commit message: Add files via upload
Parts:
- removed A10: 74LS194, Apple:DIP-16_W7.62mm, symbol 74xx:74LS194
- removed unit 5 of A2
- removed unit 5 of B13
- removed unit 5 of C14
- removed CT3: 5-50pf, symbol AppleII-rescue:CTRIM_Small-Device
- removed K14: VIDEO OUT, symbol Connector:Conn_Coaxial_Power
- added A10: 74LS194, Package_DIP:DIP-16_W7.62mm, symbol AppleII+:74LS194
- added unit 7 of C11
- added CT3: 5-50pF, Apple-II:COLOUR_TRIM, symbol Device:C_Trim_Differential
- added Cap47: 0.1uF, Apple-II:C_Disc_D5.0mm_W2.5mm_P5.00mm, symbol Device:C_Small
- added K14: RCA Connector, Apple-II:VIDEO, symbol Apple-II:Video
- added TP2: TestPoint, TestPoint:TestPoint_THTPad_1.5x1.5mm_Drill0.7mm, symbol Connector:TestPoint
- A2, B10, B11, B12, B13, B2, C11, C13, C14: footprint Apple:DIP-14_W7.62mm -> Package_DIP:DIP-14_W7.62mm
- A3, A8, A9, B4, B9: footprint Apple:DIP-16_W7.62mm -> Package_DIP:DIP-16_W7.62mm
- A5: footprint Apple:DIP-24_W15.24mm -> Package_DIP:DIP-24_W15.24mm
- B3: footprint Apple:DIP-8_W7.62mm -> Package_DIP:DIP-8_W7.62mm
- C13: footprint (none) -> Package_DIP:DIP-14_W7.62mm
- Cap13, Cap14: footprint (none) -> Apple-II:C_Disc_D5.0mm_W2.5mm_P5.00mm
- Cap15: renamed from C15; footprint (none) -> Apple-II:C_Disc_D5.0mm_W2.5mm_P5.00mm
- Cap2: footprint (none) -> Capacitor_THT:C_Disc_D7.0mm_W2.5mm_P5.00mm
- J18: footprint (none) -> Connector_PinHeader_2.54mm:PinHeader_1x04_P2.54mm_Vertical
- L1: footprint (none) -> Inductor_THT:L_Axial_L7.0mm_D3.3mm_P12.70mm_Horizontal_Fastron_MICC
- Q3: footprint digikey-footprints:TO-92-3 -> Package_TO_SOT_THT:TO-92
- R10, R12, R13, R5, R9: footprint (none) -> Apple-II:R_Axial_DIN0207_L6.3mm_D2.5mm_P10.16mm_Horizontal
- R11: footprint (none) -> Potentiometer_THT:Potentiometer_Bourns_3266Y_Vertical
- R6, R7, R8: footprint Resistor_THT:R_Axial_DIN0207_L6.3mm_D2.5mm_P10.16mm_Horizontal -> Apple-II:R_Axial_DIN0207_L6.3mm_D2.5mm_P10.16mm_Horizontal
Connections:
- net SOFT5a is gone; now on net SOFT5: A2.8, A3.9 (Clr), B4.1 (Mr), B4.2 (Dsr)
- net +5V: now also A10.16 (VCC), C11.14 (VCC), Cap47.2
- net 14M: now also A10.11 (Cp)
- net A3-2: now also A10.6 (P3)
- net A8-3-A9-B9: now also A8.3 (I1a), A9.13 (I6), B9.15 (Q0)
- net C14-6: now also A10.5 (P2)
- net Color_Burst: now also TP2.1
- net GND: now also A10.8 (GND), C11.7 (GND), CT3.1, Cap47.1, K14.1
- net LD194: now also A10.10 (S1), A10.9 (S0)
- net SOFT5: now also A10.1 (Mr), A10.2 (Dsr), A10.7 (Dsl)
- net at A9.10 (S1): now also A10.15 (Q0)
- net at A9.11 (S0): now also A10.14 (Q1)
- net B9-13: now reaches A9.12 (I7), B9.13 (Q2)
- net at A9.7 (~{E}): now also A10.13 (Q2)
- net at Cap2.1, L1.1, R5.2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: now also CT3.2
- net A3-1: now reaches A3.1 (Ds), B2.12
- net A3-1: now also A10.12 (Q3)
- net at R10.2: now also K14.2
- net A8-12: no longer names the net of A8.12 (Zc)
- net A8-12: now also A10.4 (P1)
- net A8-7: no longer names the net of A8.7 (Zb)
- net A8-7: now also A10.3 (P0)
- no-connect marks 6 -> 8
Other:
- note added: "Note: See RAM circuit."
- note removed: "Composite Video Output"
- note removed: "Data Selector"
- note removed: "Flashing"
- note removed: "Graphics Shift Register"
- note removed: "H[0..5]"
- note removed: "Inverse Video"
- note removed: "LD6"
- note removed: "LD7"
- note removed: "Note: See Data Latch."
- note removed: "Shift Register"
- note removed: "Shift Register Configuration"
- note removed: "V[0..5]"
- moved on the sheet: A8, B11B, B12B, B13D, Cap13, Cap14, J18, R10, R11

Commit message: Add files via upload
Parts:
- TP2: footprint TestPoint:TestPoint_THTPad_1.5x1.5mm_Drill0.7mm -> Apple-II:TestPoint
Changed lines of the file:
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@@
       (effects (font (size 1.27 1.27)))
     )
-    (property "Footprint" "TestPoint:TestPoint_THTPad_1.5x1.5mm_Drill0.7mm" (at 173.99 117.094 0)
+    (property "Footprint" "Apple-II:TestPoint" (at 173.99 117.094 0)
       (effects (font (size 1.27 1.27)) hide)
     )
