File: RAMAddressMux.kicad_sch (KiCad schematic)
At the start: 18 parts, among them J1 74LS257

Commit message: Add files via upload
Other:
- note added: "Video Memory: Text P1 $400 $7FF Text P2 $800 $BFF Low Res P1 $400 $7FF Low Res P2 $800 $BFF Hi Res P1 $2000 $3FFF Hi Res P2 $4000 $5FFF"
- moved on the sheet: A2B, C11A, C11C, C12, C14A, C14D, D1, D2B, E1, E11, E12, E13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

Commit message: Add files via upload
Parts:
- added unit 5 of H1
Connections:
- net +5V: now also H1.14 (VCC)
- net GND: now also H1.7 (GND)
Other:
- moved on the sheet: E2C, F2C
Changed lines of the file:
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@@
   (junction (at 300.482 140.97) (diameter 0) (color 0 0 0 0)
   )
+  (junction (at 212.09 223.52) (diameter 0) (color 0 0 0 0)
+  )
   (junction (at 273.05 111.76) (diameter 0) (color 0 0 0 0)
   )
-  (junction (at 228.346 224.028) (diameter 0) (color 0 0 0 0)
-  )
   (junction (at 237.744 177.8) (diameter 0) (color 0 0 0 0)
   )
@@
   (junction (at 230.378 111.76) (diameter 0) (color 0 0 0 0)
   )
+  (junction (at 227.33 195.58) (diameter 0) (color 0 0 0 0)
+  )
   (junction (at 236.982 152.4) (diameter 0) (color 0 0 0 0)
   )
@@
   (junction (at 266.954 104.14) (diameter 0) (color 0 0 0 0)
   )
+  (junction (at 212.09 195.58) (diameter 0) (color 0 0 0 0)
+  )
   (junction (at 297.942 135.89) (diameter 0) (color 0 0 0 0)
   )
@@
   (junction (at 235.204 154.94) (diameter 0) (color 0 0 0 0)
   )
-  (junction (at 228.346 196.85) (diameter 0) (color 0 0 0 0)
-  )
   (junction (at 319.532 96.012) (diameter 0) (color 0 0 0 0)
   )
   (junction (at 236.982 122.936) (diameter 0) (color 0 0 0 0)
+  )
+  (junction (at 227.33 223.52) (diameter 0) (color 0 0 0 0)
   )
   (no_connect (at 110.236 171.196))
@@
     (stroke (width 0) (type default))
   )
-  (wire (pts (xy 228.346 224.536) (xy 228.346 224.028))
+  (wire (pts (xy 227.33 223.52) (xy 227.33 224.79))
     (stroke (width 0) (type default))
   )
@@
     (stroke (width 0) (type default))
   )
-  (wire (pts (xy 213.106 196.85) (xy 228.346 196.85))
+  (wire (pts (xy 212.09 195.58) (xy 227.33 195.58))
     (stroke (width 0) (type default))
   )
@@
     (stroke (width 0) (type default))
   )
-  (wire (pts (xy 228.346 224.028) (xy 228.346 223.012))
-    (stroke (width 0) (type default))
-  )
   (wire (pts (xy 110.236 166.116) (xy 119.126 166.116))
     (stroke (width 0) (type default))
@@
     (stroke (width 0) (type default))
   )
-  (wire (pts (xy 213.106 224.028) (xy 228.346 224.028))
+  (wire (pts (xy 196.85 223.52) (xy 212.09 223.52))
     (stroke (width 0) (type default))
   )
@@
     (stroke (width 0) (type default))
   )
-  (wire (pts (xy 213.106 197.612) (xy 213.106 196.85))
+  (wire (pts (xy 212.09 195.58) (xy 212.09 196.85))
     (stroke (width 0) (type default))
   )
@@
     (stroke (width 0) (type default))
   )
+  (wire (pts (xy 227.33 194.31) (xy 227.33 195.58))
+    (stroke (width 0) (type default))
+  )
   (wire (pts (xy 213.36 104.14) (xy 238.76 104.14))
     (stroke (width 0) (type default))
   )
-  (wire (pts (xy 213.106 223.012) (xy 213.106 224.028))
+  (wire (pts (xy 227.33 222.25) (xy 227.33 223.52))
+    (stroke (width 0) (type default))
+  )
+  (wire (pts (xy 212.09 222.25) (xy 212.09 223.52))
     (stroke (width 0) (type default))
   )
@@
     (stroke (width 0) (type default))
   )
+  (wire (pts (xy 212.09 195.58) (xy 196.85 195.58))
+    (stroke (width 0) (type default))
+  )
   (wire (pts (xy 84.836 178.816) (xy 81.026 178.816))
     (stroke (width 0) (type default))
@@
     (stroke (width 0) (type default))
   )
+  (wire (pts (xy 212.09 223.52) (xy 227.33 223.52))
+    (stroke (width 0) (type default))
+  )
   (wire (pts (xy 81.28 176.276) (xy 84.836 176.276))
     (stroke (width 0) (type default))
@@
     (stroke (width 0) (type default))
   )
+  (wire (pts (xy 196.85 195.58) (xy 196.85 196.85))
+    (stroke (width 0) (type default))
+  )
   (wire (pts (xy 82.804 75.946) (xy 82.804 47.752))
     (stroke (width 0) (type default))
@@
     (stroke (width 0) (type default))
   )
-  (wire (pts (xy 228.346 196.342) (xy 228.346 196.85))
-    (stroke (width 0) (type default))
-  )
   (wire (pts (xy 287.274 192.532) (xy 291.338 192.532))
     (stroke (width 0) (type default))
@@
     (stroke (width 0) (type default))
   )
-  (wire (pts (xy 228.346 196.85) (xy 228.346 197.612))
+  (wire (pts (xy 227.33 195.58) (xy 227.33 196.85))
     (stroke (width 0) (type default))
   )
@@
   )
   (wire (pts (xy 144.78 171.196) (xy 144.78 172.212))
+    (stroke (width 0) (type default))
+  )
+  (wire (pts (xy 196.85 222.25) (xy 196.85 223.52))
     (stroke (width 0) (type default))
   )
@@
     )
   )
-  (symbol (lib_id "74xx:74LS139") (at 228.346 210.312 0) (unit 3)
-    (in_bom yes) (on_board yes) (dnp no)
-    (property "Reference" "F2" (at 229.87 201.676 0)
+  (symbol (lib_id "74xx:74LS139") (at 227.33 209.55 0) (unit 3)
+    (in_bom yes) (on_board yes) (dnp no)
+    (property "Reference" "F2" (at 228.854 200.914 0)
       (effects (font (size 1.27 1.27)) (justify left))
     )
-    (property "Value" "74LS139" (at 228.6 218.948 0)
+    (property "Value" "74LS139" (at 227.584 218.186 0)
       (effects (font (size 1.27 1.27)) (justify left))
     )
-    (property "Footprint" "Apple:DIP-16_W7.62mm" (at 228.346 210.312 0)
-      (effects (font (size 1.27 1.27)) hide)
-    )
-    (property "Datasheet" "http://www.ti.com/lit/ds/symlink/sn74ls139a.pdf" (at 228.346 210.312 0)
+    (property "Footprint" "Apple:DIP-16_W7.62mm" (at 227.33 209.55 0)
+      (effects (font (size 1.27 1.27)) hide)
+    )
+    (property "Datasheet" "http://www.ti.com/lit/ds/symlink/sn74ls139a.pdf" (at 227.33 209.55 0)
       (effects (font (size 1.27 1.27)) hide)
     )
@@
     )
   )
-  (symbol (lib_id "74xx:74LS139") (at 213.106 210.312 0) (unit 3)
-    (in_bom yes) (on_board yes) (dnp no)
-    (property "Reference" "E2" (at 214.376 201.676 0)
+  (symbol (lib_id "74xx:74LS139") (at 212.09 209.55 0) (unit 3)
+    (in_bom yes) (on_board yes) (dnp no)
+    (property "Reference" "E2" (at 213.36 200.914 0)
       (effects (font (size 1.27 1.27)) (justify left))
     )
-    (property "Value" "74LS139" (at 213.614 218.948 0)
+    (property "Value" "74LS139" (at 212.598 218.186 0)
       (effects (font (size 1.27 1.27)) (justify left))
     )
-    (property "Footprint" "Apple:DIP-16_W7.62mm" (at 213.106 210.312 0)
-      (effects (font (size 1.27 1.27)) hide)
-    )
-    (property "Datasheet" "http://www.ti.com/lit/ds/symlink/sn74ls139a.pdf" (at 213.106 210.312 0)
+    (property "Footprint" "Apple:DIP-16_W7.62mm" (at 212.09 209.55 0)
+      (effects (font (size 1.27 1.27)) hide)
+    )
+    (property "Datasheet" "http://www.ti.com/lit/ds/symlink/sn74ls139a.pdf" (at 212.09 209.55 0)
       (effects (font (size 1.27 1.27)) hide)
     )
@@
     )
   )
-  (symbol (lib_id "power:+5V") (at 228.346 196.342 0) (unit 1)
-    (in_bom yes) (on_board yes) (dnp no)
-    (property "Reference" "#PWR0284" (at 228.346 200.152 0)
-      (effects (font (size 1.27 1.27)) hide)
-    )
-    (property "Value" "+5V" (at 226.314 193.802 0)
-      (effects (font (size 1.27 1.27)))
-    )
-    (property "Footprint" "" (at 228.346 196.342 0)
-      (effects (font (size 1.27 1.27)) hide)
-    )
-    (property "Datasheet" "" (at 228.346 196.342 0)
+  (symbol (lib_id "power:+5V") (at 227.33 194.31 0) (unit 1)
+    (in_bom yes) (on_board yes) (dnp no)
+    (property "Reference" "#PWR0284" (at 227.33 198.12 0)
+      (effects (font (size 1.27 1.27)) hide)
+    )
+    (property "Value" "+5V" (at 225.298 191.77 0)
+      (effects (font (size 1.27 1.27)))
+    )
+    (property "Footprint" "" (at 227.33 194.31 0)
+      (effects (font (size 1.27 1.27)) hide)
+    )
+    (property "Datasheet" "" (at 227.33 194.31 0)
       (effects (font (size 1.27 1.27)) hide)
     )
@@
     )
   )
-  (symbol (lib_id "power:GND") (at 228.346 224.536 0) (unit 1)
-    (in_bom yes) (on_board yes) (dnp no)
-    (property "Reference" "#PWR0285" (at 228.346 230.886 0)
-      (effects (font (size 1.27 1.27)) hide)
-    )
-    (property "Value" "GND" (at 230.632 227.33 0)
-      (effects (font (size 1.27 1.27)))
-    )
-    (property "Footprint" "" (at 228.346 224.536 0)
-      (effects (font (size 1.27 1.27)) hide)
-    )
-    (property "Datasheet" "" (at 228.346 224.536 0)
+  (symbol (lib_id "power:GND") (at 227.33 224.79 0) (unit 1)
+    (in_bom yes) (on_board yes) (dnp no)
+    (property "Reference" "#PWR0285" (at 227.33 231.14 0)
+      (effects (font (size 1.27 1.27)) hide)
+    )
+    (property "Value" "GND" (at 229.616 227.584 0)
+      (effects (font (size 1.27 1.27)))
+    )
+    (property "Footprint" "" (at 227.33 224.79 0)
+      (effects (font (size 1.27 1.27)) hide)
+    )
+    (property "Datasheet" "" (at 227.33 224.79 0)
       (effects (font (size 1.27 1.27)) hide)
     )
@@
         )
       )
+    )
+  )
+  (symbol (lib_id "74xx:74LS08") (at 196.85 209.55 0) (unit 5)
+    (in_bom yes) (on_board yes) (dnp no)
+    (property "Reference" "H1" (at 198.12 200.66 0)
+      (effects (font (size 1.27 1.27)) (justify left))
+    )
+    (property "Value" "74LS08" (at 198.12 218.44 0)
+      (effects (font (size 1.27 1.27)) (justify left))
+    )
+    (property "Footprint" "" (at 196.85 209.55 0)
+      (effects (font (size 1.27 1.27)) hide)
+    )
+    (property "Datasheet" "http://www.ti.com/lit/gpn/sn74LS08" (at 196.85 209.55 0)
+      (effects (font (size 1.27 1.27)) hide)
+    )
+    (pin "14")
+    (pin "7")
+    (pin "5")
+    (pin "11")
+    (pin "13")
+    (pin "4")
+    (pin "8")
+    (pin "9")
+    (pin "6")
+    (pin "1")
+    (pin "2")
+    (pin "3")
+    (pin "12")
+    (pin "10")
+    (instances
+      (project "AppleII"
+        (path "/f1f08369-4db3-46f7-9b89-a5d3cfbed55a/00000000-0000-0000-0000-000060210f9e"
+          (reference "H1") (unit 5)
+        )
+      )

Commit message: Add files via upload
Parts:
- added unit 3 of D2
Connections:
- net +5V: now also D2.14 (VCC)
- net GND: now also D2.7 (GND)
Other:
- moved on the sheet: E2C, F2C, H1E

Commit message: Add files via upload
Other:
- moved on the sheet: A2B, C11A, C11C, C12, C14A, C14D, D1, D2B, D2C, E1, E11, E12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

Commit message: Add files via upload
Other:
- note added: "H0"
- note added: "H1"
- note added: "H2"
- note added: "V0"
- note added: "V1"
- note added: "V2"
- moved on the sheet: A2B, C11A, C11C, C12, C14A, C14D, D1, D2B, D2C, E1, E14, E2A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

Commit message: Add files via upload
Parts:
- added unit 7 of C11
Connections:
- net +5V: now also C11.14 (VCC)
- net GND: now also C11.7 (GND)
Other:
- moved on the sheet: C14A
Changed lines of the file:
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@@
     (comment 1 "Captured from the Apple II Reference Manual (1979)")
   )
+  (junction (at 346.71 218.44) (diameter 0) (color 0 0 0 0)
+  )
   (junction (at 317.5 128.27) (diameter 0) (color 0 0 0 0)
   )
@@
   (junction (at 105.41 19.05) (diameter 0) (color 0 0 0 0)
   )
+  (junction (at 346.71 246.38) (diameter 0) (color 0 0 0 0)
+  )
   (junction (at 266.7 154.94) (diameter 0) (color 0 0 0 0)
   )
@@
     (stroke (width 0) (type default))
   )
+  (wire (pts (xy 331.47 246.38) (xy 346.71 246.38))
+    (stroke (width 0) (type default))
+  )
   (wire (pts (xy 266.7 154.94) (xy 273.05 154.94))
     (stroke (width 0) (type default))
@@
     (stroke (width 0) (type default))
   )
+  (wire (pts (xy 346.71 218.44) (xy 331.47 218.44))
+    (stroke (width 0) (type default))
+  )
   (wire (pts (xy 107.95 210.82) (xy 133.35 210.82))
     (stroke (width 0) (type default))
@@
     (stroke (width 0) (type default))
   )
+  (wire (pts (xy 331.47 245.11) (xy 331.47 246.38))
+    (stroke (width 0) (type default))
+  )
   (wire (pts (xy 335.28 125.73) (xy 349.25 125.73))
     (stroke (width 0) (type default))
@@
     (stroke (width 0) (type default))
   )
+  (wire (pts (xy 331.47 218.44) (xy 331.47 219.71))
+    (stroke (width 0) (type default))
+  )
   (wire (pts (xy 38.1 165.1) (xy 66.04 165.1))
     (stroke (width 0) (type default))
@@
     )
   )
-  (symbol (lib_id "74xx:74LS32") (at 306.07 233.68 0) (mirror x) (unit 1)
+  (symbol (lib_id "74xx:74LS32") (at 255.27 231.14 0) (mirror x) (unit 1)
     (in_bom yes) (on_board yes) (dnp no)
-    (property "Reference" "C14" (at 304.292 227.076 0)
+    (property "Reference" "C14" (at 253.492 224.536 0)
       (effects (font (size 1.27 1.27)))
     )
-    (property "Value" "74LS32" (at 305.816 228.854 0)
+    (property "Value" "74LS32" (at 255.016 226.314 0)
       (effects (font (size 1.27 1.27)))
     )
-    (property "Footprint" "Apple:DIP-14_W7.62mm" (at 306.07 233.68 0)
+    (property "Footprint" "Apple:DIP-14_W7.62mm" (at 255.27 231.14 0)
       (effects (font (size 1.27 1.27)) hide)
     )
-    (property "Datasheet" "http://www.ti.com/lit/gpn/sn74LS32" (at 306.07 233.68 0)
+    (property "Datasheet" "http://www.ti.com/lit/gpn/sn74LS32" (at 255.27 231.14 0)
       (effects (font (size 1.27 1.27)) hide)
     )
@@
         )
       )
+    )
+  )
+  (symbol (lib_id "74xx:74LS04") (at 331.47 232.41 0) (unit 7)
+    (in_bom yes) (on_board yes) (dnp no)
+    (property "Reference" "C11" (at 332.74 223.52 0)
+      (effects (font (size 1.27 1.27)) (justify left))
+    )
+    (property "Value" "74LS04" (at 332.74 241.3 0)
+      (effects (font (size 1.27 1.27)) (justify left))
+    )
+    (property "Footprint" "" (at 331.47 232.41 0)
+      (effects (font (size 1.27 1.27)) hide)
+    )
+    (property "Datasheet" "http://www.ti.com/lit/gpn/sn74LS04" (at 331.47 232.41 0)
+      (effects (font (size 1.27 1.27)) hide)
+    )
+    (pin "14")
+    (pin "5")
+    (pin "3")
+    (pin "8")
+    (pin "6")
+    (pin "9")
+    (pin "13")
+    (pin "10")
+    (pin "4")
+    (pin "12")
+    (pin "2")
+    (pin "7")
+    (pin "1")
+    (pin "11")
+    (instances
+      (project "AppleII"
+        (path "/f1f08369-4db3-46f7-9b89-a5d3cfbed55a/00000000-0000-0000-0000-000060210f9e"
+          (reference "C11") (unit 7)
+        )
+      )

Commit message: Add files via upload
Changed lines of the file:
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@@
   )
   (text "Video Memory:\nText P1		$400	$7FF\nText P2		$800	$BFF\nLow Res P1	$400	$7FF\nLow Res P2	$800	$BFF\nHi Res P1	$2000	$3FFF\nHi Res P2	$4000	$5FFF"
-    (at 374.65 34.29 0)
+    (at 367.03 39.37 0)
     (effects (font (size 1.27 1.27)) (justify left bottom))
   )

Commit message: Add files via upload
Parts:
- removed unit 7 of C11
- removed RA2, RA3: 1K, Resistor_THT:R_Array_SIP8, symbol Device:R_Network07_US
- added unit 5 of C14
- added Cap17, Cap41, Cap44, Cap49: 0.1uF, Apple-II:C_Disc_D5.0mm_W2.5mm_P5.00mm, symbol Device:C_Small
- added RA02, RA03: 1K, Resistor_THT:R_Array_SIP8, symbol Device:R_Network07_US
- added TP1: TestPoint, TestPoint:TestPoint_THTPad_1.5x1.5mm_Drill0.7mm, symbol Connector:TestPoint
- A2, C11, C14, D1, D2, E1, F1, H1: footprint Apple:DIP-14_W7.62mm -> Package_DIP:DIP-14_W7.62mm
- C12, E11, E12, E13, E14, E2, F2, J1: footprint Apple:DIP-16_W7.62mm -> Package_DIP:DIP-16_W7.62mm
- D2, H1: footprint (none) -> Package_DIP:DIP-14_W7.62mm
Connections:
- net +5V: now also C14.14 (VCC), Cap17.2, Cap41.2, Cap44.2, Cap49.2, RA02.1 (common)
- net GND: now also C14.7 (GND), Cap17.1, Cap41.1, Cap44.1, Cap49.1, RA03.1 (common)
- net RA0: now also RA02.7 (R6), RA03.7 (R6)
- net RA1: now also RA02.5 (R4), RA03.5 (R4)
- net RA2: now also RA02.3 (R2), RA03.3 (R2)
- net RA3: now also RA02.8 (R7), RA03.8 (R7)
- net RA4: now also RA02.6 (R5), RA03.6 (R5)
- net RA5: now also RA02.4 (R3), RA03.4 (R3)
- net at D1.1, E1.1, E2.4 (O0): now also TP1.1
- no-connect marks 4 -> 9
Other:
- note removed: "H0"
- note removed: "H1"
- note removed: "H2"
- note removed: "V0"
- note removed: "V1"
- note removed: "V2"
- moved on the sheet: A2B, C11A, C11C, C12, C14A, C14D, D1, D2B, E1, E11, E12, E13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
