File: RAMAddressMux.kicad_sch (KiCad schematic)
At the start: 23 parts, among them J1 74LS257

Commit message: Add files via upload
Parts:
- TP1: footprint TestPoint:TestPoint_THTPad_1.5x1.5mm_Drill0.7mm -> Apple-II:TestPoint
Changed lines of the file:
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@@
       (effects (font (size 1.27 1.27)) (justify left))
     )
-    (property "Footprint" "TestPoint:TestPoint_THTPad_1.5x1.5mm_Drill0.7mm" (at 272.034 89.408 0)
+    (property "Footprint" "Apple-II:TestPoint" (at 272.034 89.408 0)
       (effects (font (size 1.27 1.27)) hide)
     )
