File: AppleII.kicad_pcb (KiCad board)
At the start: 2 copper layers, 215.5 x 361.2 mm, 204 parts, among them J0 Cassette Data In, J1 74LS257, J13 74LS74, J14 GAME_IO_Conn, J18 Aux Video, J2 Cassette Data Out, J3 Conn_01x16, J4 Conn_01x25, J5 Conn_01x25, J6 Conn_01x24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

Commit message: Add files via upload
Parts:
- J3: footprint Connector_PinHeader_2.54mm:PinHeader_1x16_P2.54mm_Vertical -> Apple-II:Keyboard Connector 16 Pin
- JP-User1: footprint Connector_PinSocket_2.54mm:PinSocket_1x02_P2.54mm_Vertical -> Apple-II:User-1
- SPKR1: footprint Connector_PinSocket_2.54mm:PinSocket_1x02_P2.54mm_Vertical -> Connector_PinHeader_2.54mm:PinHeader_1x02_P2.54mm_Vertical
- TP1, TP2: footprint TestPoint:TestPoint_THTPad_1.5x1.5mm_Drill0.7mm -> Apple-II:TestPoint
