File: AppleII.kicad_pcb (KiCad board)
At the start: 2 copper layers, 215.5 x 361.2 mm, 204 parts, among them J0 Cassette Data In, J1 74LS257, J13 74LS74, J14 GAME_IO_Conn, J18 Aux Video, J2 Cassette Data Out, J3 Conn_01x16, J4 Conn_01x25, J5 Conn_01x25, J6 Conn_01x24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

Commit message: Add files via upload
Parts:
- H7: value locked -> 6502
Other:
- board text added: "1"
- board text added: "1.5K"
- board text added: "10"
- board text added: "100"
- board text added: "11"
- board text added: "12"
- board text added: "12K"
- board text added: "13"
- board text added: "14"
- board text added: "2"
- board text added: "2.0K"
- board text added: "2.7K"
- board text added: "200"
- board text added: "220K"
- board text added: "27"
- board text added: "27uH"
- board text added: "2N3904"
- board text added: "3"
- board text added: "4"
- board text added: "47K"
- board text added: "47pF"
- board text added: "5"
- board text added: "6"
- board text added: "7"
- board text added: "741C"
- board text added: "74LS257"
- board text added: "74LS74"
- board text added: "8"
- board text added: "9"
- board text added: "A"
- board text added: "B"
- board text added: "C"
- board text added: "COLOR TRIM"
- board text added: "D"
- board text added: "E"
- board text added: "F"
- board text added: "GAME I/O"
- board text added: "H"
- board text added: "IN"
- board text added: "IN914"
- board text added: "J"
- board text added: "K"
- board text added: "MEMORY SELECT"
- board text added: "MPSA13"
- board text added: "OUT"
- board text added: "POWER"
- board text added: "VIDEO"
- board text removed: "locked"

Commit message: Add files via upload
Parts:
- removed the G*** at (143.4, 141.8)
- added G***: LOGO, Apple-II:logo2, F.Cu at (143.3, 140.7)
- added G***: LOGO, Apple-II:copyright, F.Cu at (129.7, 145.7)
Other:
- board text added: "1977"
