File: IO_AddressDecode.kicad_sch (KiCad schematic)
At the start: 35 parts, among them J0 Cassette Data In, J13 74LS74, J14 GAME_IO_Conn, J2 Cassette Data Out, K13 MA741, Q4 MPSA13

Commit message: Add files via upload
Parts:
- added A1: Keyboard_Connector, Apple:DIP-16_W7.62mm, symbol AppleII+:AppleII+_Keyboard_Connector
- added B10: 74LS74, Apple:DIP-14_W7.62mm, symbol 74xx:74LS74
- added F3: 74LS138, Apple:DIP-16_W7.62mm, symbol 74xx:74LS138
- added H1: 74LS08, Apple:DIP-14_W7.62mm, symbol 74xx:74LS08
Connections:
- net +5V: now also A1.1 (+5V), F3.16 (VCC)
- net GND: now also H12.8 (GND), A1.8 (GND), F3.8 (GND)
- net PHI1: now also F3.4 (E1), F3.5 (E2)
- net ~{C000-C7FF}: now also F3.15 (O0)
- net ~{CLR_STB}: now also B10.13 (~{R})
- new net: F3.6 (E3), H1.6
- new net: A1.2 (STROBE), B10.11 (C)
- new net -12V: A1.15 (-12V)
- new net A11: F3.1 (A0)
- new net A12: F3.2 (A1)
- new net A13: F3.3 (A2)
- new net A14: H1.4
- new net A15: H1.5
- new net KBD_Data0: A1.12 (Data0)
- new net KBD_Data1: A1.13 (Data1)
- new net KBD_Data2: A1.10 (Data2)
- new net KBD_Data3: A1.11 (Data3)
- new net KBD_Data4: A1.6 (Data4)
- new net KBD_Data5: A1.5 (Data5)
- new net KBD_Data6: A1.7 (Data6)
- new net KBD_STB: B10.9 (Q)
- new net ROM_Select_D0: F3.13 (O2)
- new net ROM_Select_D8: F3.12 (O3)
- new net ROM_Select_E0: F3.11 (O4)
- new net ROM_Select_E8: F3.10 (O5)
- new net ROM_Select_F0: F3.9 (O6)
- new net ROM_Select_F8: F3.7 (O7)
- new net ~{IO_STB}: F3.14 (O1)
- new net ~{RESET}: A1.3 (~{RESET})
- no-connect marks 4 -> 5
Other:
- note added: "Address Decoder"
- note added: "C000"
- note added: "C000-C7FF - to I/O Selects and Device Selects"
- note added: "C010"
- note added: "C020"
- note added: "C030"
- note added: "C040"
- note added: "C050"
- note added: "C050/C051"
- note added: "C052/C053"
- note added: "C054/C055"
- note added: "C056/C057"
- note added: "C058/C059"
- note added: "C05A/C05B"
- note added: "C05C/C05D"
- note added: "C05E/C05F"
- note added: "C060"
- note added: "C061"
- note added: "C062"
- note added: "C063"
- note added: "C064"
- note added: "C065"
- note added: "C066"
- note added: "C067"
- note added: "C070"
- note added: "IO Strobe - Goes low to all Peripheral Connectors (slots) when accessing address ranges C800-C8FF"
- note added: "Onboard I/O"
- moved on the sheet: CR1, Cap10, Cap11, Cap12, Cap5, Cap6, Cap7, Cap8, Cap9, F13, F14, H12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

Commit message: Add files via upload
Parts:
- renumbered A1 to A7, F3 to F12
Changed lines of the file:
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@@
   )
   (text "IO Strobe - Goes low to all \nPeripheral Connectors (slots)\nwhen accessing address ranges\nC800-C8FF"
-    (at 101.6 69.85 0)
+    (at 97.79 72.39 0)
     (effects (font (size 1.27 1.27)) (justify left bottom))
   )
@@
     (effects (font (size 1.27 1.27) (thickness 0.254) bold) (justify left bottom))
   )
-  (text "C061" (at 203.2 106.68 0)
+  (text "C061" (at 182.88 106.68 0)
     (effects (font (size 1.27 1.27)) (justify left bottom))
   )
@@
     (effects (font (size 1.27 1.27) (thickness 0.254) bold) (justify left bottom))
   )
-  (text "C062" (at 203.2 104.14 0)
+  (text "C062" (at 182.88 104.14 0)
     (effects (font (size 1.27 1.27)) (justify left bottom))
   )
@@
     (effects (font (size 1.27 1.27)) (justify left bottom))
   )
-  (text "C060" (at 203.2 109.22 0)
+  (text "C060" (at 182.88 109.22 0)
     (effects (font (size 1.27 1.27)) (justify left bottom))
   )
@@
   (symbol (lib_id "AppleII+:AppleII+_Keyboard_Connector") (at 251.46 171.45 0) (unit 1)
     (in_bom yes) (on_board yes) (dnp no)
-    (property "Reference" "A1" (at 251.46 160.02 0)
+    (property "Reference" "A7" (at 251.46 160.02 0)
       (effects (font (size 1.27 1.27)))
     )
@@
       (project "AppleII"
         (path "/f1f08369-4db3-46f7-9b89-a5d3cfbed55a/00000000-0000-0000-0000-00006017a131"
-          (reference "A1") (unit 1)
+          (reference "A7") (unit 1)
         )
       )
@@
   (symbol (lib_id "74xx:74LS138") (at 63.5 67.31 0) (unit 1)
     (in_bom yes) (on_board yes) (dnp no)
-    (property "Reference" "F3" (at 69.596 54.102 0)
+    (property "Reference" "F12" (at 69.596 54.102 0)
       (effects (font (size 1.27 1.27)))
     )
@@
       (project "AppleII"
         (path "/f1f08369-4db3-46f7-9b89-a5d3cfbed55a/00000000-0000-0000-0000-00006017a131"
-          (reference "F3") (unit 1)
-        )
-      )
+          (reference "F12") (unit 1)
+        )
+      )

Commit message: Add files via upload
Connections:
- net ROM_Select_D0 renamed ROM-SELECT-D0
- net ROM_Select_D8 renamed ROM-SELECT-D8
- net ROM_Select_E0 renamed ROM-SELECT-E0
- net ROM_Select_E8 renamed ROM-SELECT-E8
- net ROM_Select_F0 renamed ROM-SELECT-F0
- net ROM_Select_F8 renamed ROM-SELECT-F8
- net Soft5 renamed SOFT5
- net ~{IO-Select-1} renamed ~{IO-SELECT-1}
- net ~{IO-Select-2} renamed ~{IO-SELECT-2}
- net ~{IO-Select-3} renamed ~{IO-SELECT-3}
- net ~{IO-Select-4} renamed ~{IO-SELECT-4}
- net ~{IO-Select-5} renamed ~{IO-SELECT-5}
- net ~{IO-Select-6} renamed ~{IO-SELECT-6}
- net ~{IO-Select-7} renamed ~{IO-SELECT-7}
Other:
- note added: "Note: Pin 6 is shown grounded on the PCB."
Changed lines of the file:
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@@
+    (stroke (width 0) (type default))
+  )
+  (wire (pts (xy 76.2 77.47) (xy 81.28 77.47))
     (stroke (width 0) (type default))
   )
@@
     (stroke (width 0) (type default))
   )
-  (wire (pts (xy 76.2 69.85) (xy 90.424 69.85))
-    (stroke (width 0) (type default))
-  )
   (bus (pts (xy 58.42 115.57) (xy 58.42 118.11))
     (stroke (width 0) (type default))
@@
     (stroke (width 0) (type default))
   )
+  (wire (pts (xy 76.2 72.39) (xy 81.28 72.39))
+    (stroke (width 0) (type default))
+  )
   (wire (pts (xy 66.04 133.35) (xy 63.5 133.35))
     (stroke (width 0) (type default))
@@
     (stroke (width 0) (type default))
   )
-  (wire (pts (xy 76.2 72.39) (xy 90.424 72.39))
-    (stroke (width 0) (type default))
-  )
   (wire (pts (xy 311.15 233.68) (xy 304.8 233.68))
     (stroke (width 0) (type default))
@@
     (stroke (width 0) (type default))
   )
-  (wire (pts (xy 76.2 67.31) (xy 90.424 67.31))
-    (stroke (width 0) (type default))
-  )
   (wire (pts (xy 323.85 177.8) (xy 323.85 186.69))
     (stroke (width 0) (type default))
@@
     (stroke (width 0) (type default))
   )
-  (wire (pts (xy 76.2 77.47) (xy 90.424 77.47))
-    (stroke (width 0) (type default))
-  )
   (wire (pts (xy 383.286 94.996) (xy 385.826 94.996))
     (stroke (width 0) (type default))
@@
     (stroke (width 0) (type default))
   )
+  (wire (pts (xy 76.2 74.93) (xy 81.28 74.93))
+    (stroke (width 0) (type default))
+  )
   (wire (pts (xy 302.26 186.69) (xy 308.61 186.69))
     (stroke (width 0) (type default))
@@
     (stroke (width 0) (type default))
   )
-  (wire (pts (xy 76.2 64.77) (xy 90.424 64.77))
-    (stroke (width 0) (type default))
-  )
   (bus (pts (xy 187.96 63.5) (xy 187.96 78.74))
     (stroke (width 0) (type default))
@@
     (stroke (width 0) (type default))
   )
+  (wire (pts (xy 76.2 67.31) (xy 81.28 67.31))
+    (stroke (width 0) (type default))
+  )
   (wire (pts (xy 336.55 200.914) (xy 331.47 200.914))
     (stroke (width 0) (type default))
@@
     (stroke (width 0) (type default))
   )
-  (wire (pts (xy 76.2 74.93) (xy 90.424 74.93))
-    (stroke (width 0) (type default))
-  )
   (wire (pts (xy 25.4 69.85) (xy 29.972 69.85))
     (stroke (width 0) (type default))
@@
     (stroke (width 0) (type default))
   )
+  (wire (pts (xy 76.2 69.85) (xy 81.28 69.85))
+    (stroke (width 0) (type default))
+  )
   (wire (pts (xy 328.93 223.52) (xy 317.5 223.52))
     (stroke (width 0) (type default))
@@
   )
   (wire (pts (xy 156.21 50.8) (xy 156.21 53.34))
+    (stroke (width 0) (type default))
+  )
+  (wire (pts (xy 76.2 64.77) (xy 81.28 64.77))
     (stroke (width 0) (type default))
   )
@@
     (effects (font (size 1.27 1.27)) (justify left bottom))
   )
+  (text "Note:  Pin 6 is shown\ngrounded on the PCB." (at 153.67 124.46 0)
+    (effects (font (size 1.27 1.27)) (justify left bottom))
+  )
   (text "C070" (at 207.01 50.8 0)
     (effects (font (size 1.27 1.27)) (justify left bottom))
@@
   )
   (text "IO Strobe - Goes low to all \nPeripheral Connectors (slots)\nwhen accessing address ranges\nC800-C8FF"
-    (at 97.79 72.39 0)
+    (at 100.33 68.58 0)
     (effects (font (size 1.27 1.27)) (justify left bottom))
   )
@@
     (effects (font (size 1.27 1.27)) (justify left bottom))
   )
-  (label "ROM_Select_E0" (at 76.2 69.85 0) (fields_autoplaced)
-    (effects (font (size 1.27 1.27)) (justify left bottom))
-  )
   (label "GamePort_ANN2" (at 345.186 135.89 0) (fields_autoplaced)
     (effects (font (size 1.27 1.27)) (justify left bottom))
@@
     (effects (font (size 1.27 1.27)) (justify left bottom))
   )
-  (label "ROM_Select_E8" (at 76.2 72.39 0) (fields_autoplaced)
-    (effects (font (size 1.27 1.27)) (justify left bottom))
-  )
   (label "A7" (at 26.162 182.88 0) (fields_autoplaced)
-    (effects (font (size 1.27 1.27)) (justify left bottom))
-  )
-  (label "ROM_Select_D8" (at 76.2 67.31 0) (fields_autoplaced)
     (effects (font (size 1.27 1.27)) (justify left bottom))
   )
@@
     (effects (font (size 1.27 1.27)) (justify right bottom))
   )
-  (label "ROM_Select_F8" (at 76.2 77.47 0) (fields_autoplaced)
-    (effects (font (size 1.27 1.27)) (justify left bottom))
-  )
   (label "GamePort_ANN0" (at 345.186 130.81 0) (fields_autoplaced)
     (effects (font (size 1.27 1.27)) (justify left bottom))
@@
     (effects (font (size 1.27 1.27)) (justify right bottom))
   )
-  (label "ROM_Select_D0" (at 76.2 64.77 0) (fields_autoplaced)
-    (effects (font (size 1.27 1.27)) (justify left bottom))
-  )
   (label "A13" (at 25.654 64.77 0) (fields_autoplaced)
     (effects (font (size 1.27 1.27)) (justify left bottom))
@@
     (effects (font (size 1.27 1.27)) (justify left bottom))
   )
-  (label "ROM_Select_F0" (at 76.2 74.93 0) (fields_autoplaced)
-    (effects (font (size 1.27 1.27)) (justify left bottom))
-  )
   (label "A3" (at 316.23 40.64 0) (fields_autoplaced)
     (effects (font (size 1.27 1.27)) (justify left bottom))
@@
     (property "Intersheetrefs" "${INTERSHEET_REFS}" (at 359.41 33.02 0)
       (effects (font (size 1.27 1.27)) hide)
+    )
+  )
+  (global_label "ROM-SELECT-D0" (shape output) (at 81.28 64.77 0) (fields_autoplaced)
+    (effects (font (size 1.27 1.27)) (justify left))
+    (property "Intersheetrefs" "${INTERSHEET_REFS}" (at 100.0604 64.77 0)
+      (effects (font (size 1.27 1.27)) (justify left) hide)
     )
   )
@@
     )
   )
-  (global_label "~{IO-Select-4}" (shape output) (at 106.68 125.73 0)
+  (global_label "~{IO-SELECT-4}" (shape output) (at 106.68 125.73 0)
     (effects (font (size 1.27 1.27)) (justify left))
     (property "Intersheetrefs" "${INTERSHEET_REFS}" (at 106.68 125.73 0)
@@
     )
   )
-  (global_label "~{IO-Select-6}" (shape output) (at 106.68 130.81 0)
+  (global_label "ROM-SELECT-E0" (shape output) (at 81.28 69.85 0) (fields_autoplaced)
+    (effects (font (size 1.27 1.27)) (justify left))
+    (property "Intersheetrefs" "${INTERSHEET_REFS}" (at 99.9394 69.85 0)
+      (effects (font (size 1.27 1.27)) (justify left) hide)
+    )
+  )
+  (global_label "~{IO-SELECT-6}" (shape output) (at 106.68 130.81 0)
     (effects (font (size 1.27 1.27)) (justify left))
     (property "Intersheetrefs" "${INTERSHEET_REFS}" (at 106.68 130.81 0)
@@
     )
   )
+  (global_label "ROM-SELECT-D8" (shape output) (at 81.28 67.31 0) (fields_autoplaced)
+    (effects (font (size 1.27 1.27)) (justify left))
+    (property "Intersheetrefs" "${INTERSHEET_REFS}" (at 100.0604 67.31 0)
+      (effects (font (size 1.27 1.27)) (justify left) hide)
+    )
+  )
   (global_label "~{DEV-SEL-2}" (shape output) (at 91.44 175.26 0)
     (effects (font (size 1.27 1.27)) (justify left))
@@
     (property "Intersheetrefs" "${INTERSHEET_REFS}" (at 77.47 187.96 0)
       (effects (font (size 1.27 1.27)) hide)
+    )
+  )
+  (global_label "ROM-SELECT-F8" (shape output) (at 81.28 77.47 0) (fields_autoplaced)
+    (effects (font (size 1.27 1.27)) (justify left))
+    (property "Intersheetrefs" "${INTERSHEET_REFS}" (at 99.879 77.47 0)
+      (effects (font (size 1.27 1.27)) (justify left) hide)
     )
   )
@@
     )
   )
-  (global_label "~{IO-Select-5}" (shape output) (at 92.71 128.27 0)
+  (global_label "~{IO-SELECT-5}" (shape output) (at 92.71 128.27 0)
     (effects (font (size 1.27 1.27)) (justify left))
     (property "Intersheetrefs" "${INTERSHEET_REFS}" (at 92.71 128.27 0)
@@
     )
   )
-  (global_label "Soft5" (shape input) (at 302.26 186.69 180)
+  (global_label "SOFT5" (shape input) (at 302.26 186.69 180)
     (effects (font (size 1.27 1.27)) (justify right))
     (property "Intersheetrefs" "${INTERSHEET_REFS}" (at 302.26 186.69 0)
@@
     )
   )
-  (global_label "~{IO-Select-1}" (shape output) (at 92.71 118.11 0)
+  (global_label "~{IO-SELECT-1}" (shape output) (at 92.71 118.11 0)
     (effects (font (size 1.27 1.27)) (justify left))
     (property "Intersheetrefs" "${INTERSHEET_REFS}" (at 92.71 118.11 0)
@@
     )
   )
-  (global_label "Soft5" (shape input) (at 316.23 50.8 180)
+  (global_label "SOFT5" (shape input) (at 316.23 50.8 180)
     (effects (font (size 1.27 1.27)) (justify right))
     (property "Intersheetrefs" "${INTERSHEET_REFS}" (at 316.23 50.8 0)
@@
     )
   )
-  (global_label "~{IO-Select-3}" (shape output) (at 92.71 123.19 0)
+  (global_label "~{IO-SELECT-3}" (shape output) (at 92.71 123.19 0)
     (effects (font (size 1.27 1.27)) (justify left))
     (property "Intersheetrefs" "${INTERSHEET_REFS}" (at 92.71 123.19 0)
@@
     )
   )
+  (global_label "ROM-SELECT-E8" (shape output) (at 81.28 72.39 0) (fields_autoplaced)
+    (effects (font (size 1.27 1.27)) (justify left))
+    (property "Intersheetrefs" "${INTERSHEET_REFS}" (at 99.9394 72.39 0)
+      (effects (font (size 1.27 1.27)) (justify left) hide)
+    )
+  )
   (global_label "PHI0" (shape input) (at 142.24 45.72 180)
     (effects (font (size 1.27 1.27)) (justify right))
@@
     )
   )
-  (global_label "~{IO-Select-2}" (shape output) (at 106.68 120.65 0)
+  (global_label "ROM-SELECT-F0" (shape output) (at 81.28 74.93 0) (fields_autoplaced)
+    (effects (font (size 1.27 1.27)) (justify left))
+    (property "Intersheetrefs" "${INTERSHEET_REFS}" (at 99.879 74.93 0)
+      (effects (font (size 1.27 1.27)) (justify left) hide)
+    )
+  )
+  (global_label "~{IO-SELECT-2}" (shape output) (at 106.68 120.65 0)
     (effects (font (size 1.27 1.27)) (justify left))
     (property "Intersheetrefs" "${INTERSHEET_REFS}" (at 106.68 120.65 0)
@@
     )
   )
-  (global_label "~{IO-Select-7}" (shape output) (at 92.71 133.35 0)
+  (global_label "~{IO-SELECT-7}" (shape output) (at 92.71 133.35 0)
     (effects (font (size 1.27 1.27)) (justify left))
     (property "Intersheetrefs" "${INTERSHEET_REFS}" (at 92.71 133.35 0)

Commit message: Add files via upload
Connections:
- net SOFT5: now also B10.10 (~{S})
- no-connect marks 5 -> 6
Changed lines of the file:
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@@
   )
   (no_connect (at 255.27 203.2))
+  (no_connect (at 240.03 198.12))
   (no_connect (at 316.23 241.3))
   (no_connect (at 156.21 106.68))
@@
     (stroke (width 0) (type default))
   )
+  (wire (pts (xy 250.19 190.5) (xy 247.65 190.5))
+    (stroke (width 0) (type default))
+  )
   (bus (pts (xy 312.42 33.02) (xy 312.42 35.56))
     (stroke (width 0) (type default))
@@
   )
   (wire (pts (xy 181.61 35.56) (xy 195.58 35.56))
+    (stroke (width 0) (type default))
+  )
+  (wire (pts (xy 247.65 190.5) (xy 247.65 193.04))
     (stroke (width 0) (type default))
   )
@@
     )
   )
+  (global_label "SOFT5" (shape input) (at 250.19 190.5 0)
+    (effects (font (size 1.27 1.27)) (justify left))
+    (property "Intersheetrefs" "${INTERSHEET_REFS}" (at 250.19 190.5 0)
+      (effects (font (size 1.27 1.27)) hide)
+    )
+  )

Commit message: Add files via upload
Connections:
- net ~{RESET} renamed ~{RST}
Changed lines of the file:
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@@
     )
   )
-  (global_label "~{RESET}" (shape input) (at 237.236 167.64 180)
+  (global_label "~{RST}" (shape input) (at 237.236 167.64 180)
     (effects (font (size 1.27 1.27)) (justify right))
     (property "Intersheetrefs" "${INTERSHEET_REFS}" (at 237.236 167.64 0)

Commit message: Add files via upload
Connections:
- net KBD_Data0 renamed KBD0
- net KBD_Data1 renamed KBD1
- net KBD_Data2 renamed KBD2
- net KBD_Data3 renamed KBD3
- net KBD_Data4 renamed KBD4
- net KBD_Data5 renamed KBD5
- net KBD_Data6 renamed KBD6

Commit message: Add files via upload
Parts:
- removed J0: Cassette Data In, symbol AppleII-rescue:AudioJack2-Connector
- removed J2: Cassette Data Out, symbol AppleII-rescue:AudioJack2-Connector
- added Cap16, Cap18, Cap19: 0.1uF, Apple-II:C_Disc_D5.0mm_W2.5mm_P5.00mm, symbol Device:C_Small
- added J0: Cassette Data In, Apple-II:AUDIO_mono, symbol Connector_Audio:AudioJack2_Ground
- added J2: Cassette Data Out, Apple-II:AUDIO_mono, symbol Connector_Audio:AudioJack2_Ground
- added J3: Conn_01x16, Connector_PinHeader_2.54mm:PinHeader_1x16_P2.54mm_Vertical, symbol Connector_Generic:Conn_01x16
- A7, J14: footprint Apple:DIP-16_W7.62mm -> Package_DIP:DIP-16_W7.62mm_Socket_LongPads
- B10, H1, J13: footprint Apple:DIP-14_W7.62mm -> Package_DIP:DIP-14_W7.62mm
- CR1: footprint (none) -> Diode_THT:D_DO-15_P10.16mm_Horizontal
- Cap10, Cap11, Cap12, Cap5, Cap6, Cap7, Cap8, Cap9: footprint (none) -> Apple-II:C_Disc_D5.0mm_W2.5mm_P5.00mm
- F12, F13, F14, H12, H13, H14, H2: footprint Apple:DIP-16_W7.62mm -> Package_DIP:DIP-16_W7.62mm
- JP-User1: footprint (none) -> Connector_PinSocket_2.54mm:PinSocket_1x02_P2.54mm_Vertical; now not fitted
- K13: footprint Apple:DIP-8_W7.62mm -> Package_DIP:DIP-8_W7.62mm
- Q4: footprint (none) -> Package_TO_SOT_THT:TO-92; Alt (none) -> KSP13; DigiKey (none) -> KSP13BU-ND
- R15, R16, R17, R18, R19, R20, R21, R22, R23, R24, R25, R29: footprint Resistor_THT:R_Axial_DIN0207_L6.3mm_D2.5mm_P10.16mm_Horizontal -> Apple-II:R_Axial_DIN0207_L6.3mm_D2.5mm_P10.16mm_Horizontal
- SPKR1: footprint digikey-footprints:PinHeader_1x2_P2.54mm_Drill1.02mm -> Connector_PinSocket_2.54mm:PinSocket_1x02_P2.54mm_Vertical
Connections:
- net +5V: now also Cap16.2, Cap18.2, Cap19.2, J3.2 (Pin_2)
- net -12V: now also J3.3 (Pin_3)
- net GND: now also Cap16.1, Cap18.1, Cap19.1, J0.S, J2.S, J3.7 (Pin_7)
- net KBD0: now also J3.4 (Pin_4)
- net KBD1: now also J3.1 (Pin_1)
- net KBD2: now also J3.6 (Pin_6)
- net KBD3: now also J3.5 (Pin_5)
- net KBD4: now also J3.11 (Pin_11)
- net KBD5: now also J3.10 (Pin_10)
- net KBD6: now also J3.12 (Pin_12)
- net at R18.2, R19.1: now also J2.T
- net at Cap10.1: now also J0.T
- net at A7.2 (STROBE), B10.11 (C): now also J3.8 (Pin_8)
- net ROM-SELECT-D0 renamed ROM_SELECT_D0
- net ROM-SELECT-D8 renamed ROM_SELECT_D8
- net ROM-SELECT-E0 renamed ROM_SELECT_E0
- net ROM-SELECT-E8 renamed ROM_SELECT_E8
- net ROM-SELECT-F0 renamed ROM_SELECT_F0
- net ROM-SELECT-F8 renamed ROM_SELECT_F8
- net ~{RST} renamed ~{RESET}
- net ~{RESET}: now also J3.9 (Pin_9)
- no-connect marks 6 -> 12
Other:
- note removed: "Note: Pin 6 is shown grounded on the PCB."

Commit message: Add files via upload
Parts:
- J3: footprint Connector_PinHeader_2.54mm:PinHeader_1x16_P2.54mm_Vertical -> Apple-II:Keyboard Connector 16 Pin
- JP-User1: footprint Connector_PinSocket_2.54mm:PinSocket_1x02_P2.54mm_Vertical -> Apple-II:User-1
- SPKR1: footprint Connector_PinSocket_2.54mm:PinSocket_1x02_P2.54mm_Vertical -> Connector_PinHeader_2.54mm:PinHeader_1x02_P2.54mm_Vertical
Other:
- note added: "Extra Keyboard Connection?"
- moved on the sheet: J3
