File: AppleII.kicad_sch (KiCad schematic)
At the start: 0 parts

Commit message: Add files via upload
Other:
- sheet CPU renamed CPU Tranceiver Driver and Data MUX
- sheet IO_AddressDecode renamed Address Decoder and Onboard IO
- sheet RAM renamed RAM and Data Latch
- sheet Address Decoder and Onboard IO ports: added A[0..15], D[0..7]; removed none
- sheet CPU Tranceiver Driver and Data MUX ports: added A[0..15], D[0..7], LD[0..7]; removed none
- sheet Clock Generation ports: added A[0..15]; removed none
- sheet Connectors ports: added A[0..15], D[0..7]; removed none
- sheet RAM Address Multiplexing ports: added A[0..15], RA[0..5]; removed none
- sheet RAM and Data Latch ports: added LD[0..7], RA[0..5]; removed none
- sheet ROM ports: added A[0..15], D[0..7]; removed none
- sheet Video Generation ports: added LD[0..7]; removed none

Commit message: Add files via upload
Other:
- sheet Clock Generation ports: added H[0..5], V[0..5]; removed none
- sheet Video Generation ports: added H[0..5], V[0..5]; removed none
Changed lines of the file:
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@@
+    (stroke (width 0) (type default))
+  )
+  (bus (pts (xy 83.82 135.89) (xy 76.2 135.89))
     (stroke (width 0) (type default))
   )
@@
     (stroke (width 0) (type default))
   )
+  (bus (pts (xy 165.1 152.4) (xy 165.1 130.81))
+    (stroke (width 0) (type default))
+  )
+  (bus (pts (xy 177.8 135.89) (xy 170.18 135.89))
+    (stroke (width 0) (type default))
+  )
   (bus (pts (xy 64.77 101.6) (xy 140.97 101.6))
     (stroke (width 0) (type default))
@@
     (stroke (width 0) (type default))
   )
+  (bus (pts (xy 76.2 130.81) (xy 88.9 130.81))
+    (stroke (width 0) (type default))
+  )
+  (bus (pts (xy 170.18 135.89) (xy 170.18 157.48))
+    (stroke (width 0) (type default))
+  )
   (bus (pts (xy 144.78 54.61) (xy 144.78 38.1))
     (stroke (width 0) (type default))
@@
     (stroke (width 0) (type default))
   )
+  (bus (pts (xy 88.9 152.4) (xy 165.1 152.4))
+    (stroke (width 0) (type default))
+  )
   (bus (pts (xy 72.39 38.1) (xy 72.39 58.42))
     (stroke (width 0) (type default))
@@
     (stroke (width 0) (type default))
   )
+  (bus (pts (xy 88.9 130.81) (xy 88.9 152.4))
+    (stroke (width 0) (type default))
+  )
   (bus (pts (xy 64.77 50.8) (xy 140.97 50.8))
     (stroke (width 0) (type default))
@@
     (stroke (width 0) (type default))
   )
+  (bus (pts (xy 170.18 157.48) (xy 83.82 157.48))
+    (stroke (width 0) (type default))
+  )
+  (bus (pts (xy 83.82 157.48) (xy 83.82 135.89))
+    (stroke (width 0) (type default))
+  )
+  (bus (pts (xy 165.1 130.81) (xy 177.8 130.81))
+    (stroke (width 0) (type default))
+  )
   (bus (pts (xy 140.97 50.8) (xy 217.17 50.8))
     (stroke (width 0) (type default))
@@
       (effects (font (size 1.27 1.27)) (justify right))
     )
+    (pin "V[0..5]" output (at 76.2 135.89 0)
+      (effects (font (size 1.27 1.27)) (justify right))
+    )
+    (pin "H[0..5]" output (at 76.2 130.81 0)
+      (effects (font (size 1.27 1.27)) (justify right))
+    )
     (instances
       (project "AppleII"
@@
     )
   )
-  (sheet (at 177.546 127) (size 50.8 12.7) (fields_autoplaced)
-    (stroke (width 0) (type solid))
-    (fill (color 0 0 0 0.0000))
-    (property "Sheetname" "Video Generation" (at 177.546 126.2884 0)
-      (effects (font (size 1.27 1.27)) (justify left bottom))
-    )
-    (property "Sheetfile" "Video Gen.kicad_sch" (at 177.546 140.2846 0)
+  (sheet (at 177.8 127) (size 50.8 12.7) (fields_autoplaced)
+    (stroke (width 0) (type solid))
+    (fill (color 0 0 0 0.0000))
+    (property "Sheetname" "Video Generation" (at 177.8 126.2884 0)
+      (effects (font (size 1.27 1.27)) (justify left bottom))
+    )
+    (property "Sheetfile" "Video Gen.kicad_sch" (at 177.8 140.2846 0)
       (effects (font (size 1.27 1.27)) (justify left top))
     )
@@
       (effects (font (size 1.27 1.27)) (justify right))
     )
-    (instances
+    (pin "H[0..5]" input (at 177.8 130.81 180)
+      (effects (font (size 1.27 1.27)) (justify left))
+    )
+    (pin "V[0..5]" input (at 177.8 135.89 180)
+      (effects (font (size 1.27 1.27)) (justify left))
+    )
+    (instances

Commit message: Add files via upload
Other:
- sheet RAM Address Multiplexing ports: added H[0..5], V[0..5]; removed none
Changed lines of the file:
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@@
   (junction (at 144.78 54.61) (diameter 0) (color 0 0 0 0)
   )
+  (junction (at 170.18 135.89) (diameter 0) (color 0 0 0 0)
+  )
   (junction (at 68.58 54.61) (diameter 0) (color 0 0 0 0)
   )
   (junction (at 64.77 50.8) (diameter 0) (color 0 0 0 0)
   )
+  (junction (at 165.1 130.81) (diameter 0) (color 0 0 0 0)
+  )
   (junction (at 140.97 50.8) (diameter 0) (color 0 0 0 0)
   )
   (junction (at 140.97 101.6) (diameter 0) (color 0 0 0 0)
   )
+  (bus (pts (xy 170.18 135.89) (xy 170.18 86.36))
+    (stroke (width 0) (type default))
+  )
   (bus (pts (xy 148.59 58.42) (xy 148.59 109.22))
     (stroke (width 0) (type default))
@@
     (stroke (width 0) (type default))
   )
+  (bus (pts (xy 165.1 80.01) (xy 177.8 80.01))
+    (stroke (width 0) (type default))
+  )
   (bus (pts (xy 76.2 130.81) (xy 88.9 130.81))
     (stroke (width 0) (type default))
@@
     (stroke (width 0) (type default))
   )
+  (bus (pts (xy 165.1 130.81) (xy 165.1 80.01))
+    (stroke (width 0) (type default))
+  )
   (bus (pts (xy 140.97 50.8) (xy 140.97 38.1))
     (stroke (width 0) (type default))
@@
   )
   (bus (pts (xy 165.1 130.81) (xy 177.8 130.81))
+    (stroke (width 0) (type default))
+  )
+  (bus (pts (xy 170.18 86.36) (xy 177.8 86.36))
     (stroke (width 0) (type default))
   )
@@
       (effects (font (size 1.27 1.27)) (justify right))
     )
-    (instances
+    (pin "V[0..5]" input (at 177.8 86.36 180)
+      (effects (font (size 1.27 1.27)) (justify left))
+    )
+    (pin "H[0..5]" input (at 177.8 80.01 180)
+      (effects (font (size 1.27 1.27)) (justify left))
+    )
+    (instances

Commit message: Add files via upload
Other:
- sheet Address Decoder and Onboard IO ports: added KBD[0..6]; removed none
- sheet CPU Tranceiver Driver and Data MUX ports: added KBD[0..6]; removed none
Changed lines of the file:
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@@
+    (stroke (width 0) (type default))
+  )
+  (bus (pts (xy 20.32 35.56) (xy 25.4 35.56))
     (stroke (width 0) (type default))
   )
@@
   )
   (bus (pts (xy 217.17 76.2) (xy 217.17 50.8))
+    (stroke (width 0) (type default))
+  )
+  (bus (pts (xy 20.32 78.74) (xy 20.32 35.56))
     (stroke (width 0) (type default))
   )
@@
     (stroke (width 0) (type default))
   )
+  (bus (pts (xy 25.4 78.74) (xy 20.32 78.74))
+    (stroke (width 0) (type default))
+  )
   (bus (pts (xy 140.97 50.8) (xy 217.17 50.8))
     (stroke (width 0) (type default))
@@
     )
     (pin "LD[0..7]" input (at 72.39 38.1 270)
+      (effects (font (size 1.27 1.27)) (justify left))
+    )
+    (pin "KBD[0..6]" input (at 25.4 35.56 180)
       (effects (font (size 1.27 1.27)) (justify left))
     )
@@
       (effects (font (size 1.27 1.27)) (justify right))
     )
+    (pin "KBD[0..6]" output (at 25.4 78.74 180)
+      (effects (font (size 1.27 1.27)) (justify left))
+    )
     (instances

Commit message: Add files via upload
Other:
- added sheet Mounting (mounting.kicad_sch)
- added sheet Prototyping (proto.kicad_sch)
- sheet Clock Generation ports: added V[0..4]; removed V[0..5]
- sheet RAM Address Multiplexing ports: added V[0..4]; removed V[0..5]
- sheet Video Generation ports: added V[0..4]; removed V[0..5]
