File: CPU.kicad_sch (KiCad schematic)
At the start: 14 parts, among them U3 MOS6502

Commit message: Add files via upload
Parts:
- removed A7: Keyboard_Connector, Apple:DIP-16_W7.62mm, symbol AppleII+:AppleII+_Keyboard_Connector
- removed B10: 74LS74, Apple:DIP-14_W7.62mm, symbol 74xx:74LS74
Connections:
- net KBD_STB: now reaches B7.5 (I0b)
- net ~{RDY}: now reaches RA01.5 (R4), U3.2 (~{RDY})
- net ~{IRQ}: now reaches RA01.4 (R3), U3.4 (~{IRQ})
- net ~{NMI}: now reaches RA01.2 (R1), U3.6 (~{NMI})
- no-connect marks 1 -> 0
Other:
- note added: "Data MUX"
- moved on the sheet: B6, B7

Commit message: Add files via upload
Connections:
- net ~{RDY} renamed RDY
- net ~{RESET} renamed ~{RST}
- no-connect marks 0 -> 1
Other:
- note removed: "~{IRQ}"
- note removed: "~{NMI}"
- note removed: "~{RDY}"
- note removed: "~{RESET}"
- moved on the sheet: B11A, C14C, H10, H11, RA01

Commit message: Add files via upload
Connections:
- net KBD_Data0 renamed KBD0
- net KBD_Data1 renamed KBD1
- net KBD_Data2 renamed KBD2
- net KBD_Data3 renamed KBD3
- net KBD_Data4 renamed KBD4
- net KBD_Data5 renamed KBD5
- net KBD_Data6 renamed KBD6
Other:
- note added: "D[0..7]"
- note added: "KBD[0..6]"
- note added: "LD[0..7]"

Commit message: Add files via upload
Parts:
- added Cap45: 0.1uF, Apple-II:C_Disc_D5.0mm_W2.5mm_P5.00mm, symbol Device:C_Small
- B11, C11, C14: footprint Apple:DIP-14_W7.62mm -> Package_DIP:DIP-14_W7.62mm
- B6, B7, H10, H11, H3, H4, H5: footprint Apple:DIP-16_W7.62mm -> Package_DIP:DIP-16_W7.62mm
- H7: renamed from U3; value MOS6502 -> 6502; footprint Apple:DIP-40_W15.24mm -> Package_DIP:DIP-40_W15.24mm
Connections:
- net +5V: now also Cap45.2
- net GND: now also Cap45.1
- net ~{RST} renamed ~{RESET}
- no-connect marks 1 -> 0
Other:
- note removed: "D[0..7]"
- note removed: "KBD[0..6]"
- note removed: "LD[0..7]"
- moved on the sheet: B11A, C14C, H10, H11
