File: ClockGen.kicad_sch (KiCad schematic)
At the start: 21 parts, among them Q1 2N4258, Q2 2N4258, Y1 XT0001

Commit message: Add files via upload
Other:
- note added: "14.3 MHz Clock"
- note removed: "NOTE: D12, 5 & 6 are tied together."
- moved on the sheet: A2A, B1, B12C, B13C, B2A, B2B, B2C, C1, C11D, C2, Cap1, D11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

Commit message: Add files via upload
Connections:
- net SOFT5: now also D11.1 (~{MR}), D12.1 (~{MR})
- net at D12.10 (CET), D12.3 (D0), D12.5 (D2)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: no longer C11.8, D11.9 (~{PE}), D12.9 (~{PE})
- new net: C11.8, D11.9 (~{PE}), D12.9 (~{PE})
Other:
- note added: "Clock Generator"
- note added: "Video Address Generator"
- moved on the sheet: A2A, B1, B12C, B13C, B2A, B2B, B2C, C1, C11D, C2, Cap1, D11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

Commit message: Add files via upload
Parts:
- added unit 5 of B2
Connections:
- net +5V: now also B2.14 (VCC)
- net GND: now also B2.7 (GND)
Changed lines of the file:
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@@
+    (stroke (width 0) (type default))
+  )
+  (wire (pts (xy 41.91 109.22) (xy 41.91 111.76))
     (stroke (width 0) (type default))
   )
@@
   )
   (wire (pts (xy 151.13 181.61) (xy 151.13 179.07))
+    (stroke (width 0) (type default))
+  )
+  (wire (pts (xy 41.91 137.16) (xy 41.91 139.7))
     (stroke (width 0) (type default))
   )
@@
         )
       )
+    )
+  )
+  (symbol (lib_id "power:+5V") (at 41.91 109.22 0) (unit 1)
+    (in_bom yes) (on_board yes) (dnp no)
+    (property "Reference" "#PWR014" (at 41.91 113.03 0)
+      (effects (font (size 1.27 1.27)) hide)
+    )
+    (property "Value" "+5V" (at 41.91 105.41 0)
+      (effects (font (size 1.27 1.27)))
+    )
+    (property "Footprint" "" (at 41.91 109.22 0)
+      (effects (font (size 1.27 1.27)) hide)
+    )
+    (property "Datasheet" "" (at 41.91 109.22 0)
+      (effects (font (size 1.27 1.27)) hide)
+    )
+    (pin "1")
+    (instances
+      (project "AppleII"
+        (path "/f1f08369-4db3-46f7-9b89-a5d3cfbed55a/00000000-0000-0000-0000-00006016cde0"
+          (reference "#PWR014") (unit 1)
+        )
+      )
+    )
+  )
+  (symbol (lib_id "74xx:74LS86") (at 41.91 124.46 0) (unit 5)
+    (in_bom yes) (on_board yes) (dnp no)
+    (property "Reference" "B2" (at 43.18 115.57 0)
+      (effects (font (size 1.27 1.27)) (justify left))
+    )
+    (property "Value" "74LS86" (at 38.1 124.46 0)
+      (effects (font (size 1.27 1.27)) (justify left))
+    )
+    (property "Footprint" "" (at 41.91 124.46 0)
+      (effects (font (size 1.27 1.27)) hide)
+    )
+    (property "Datasheet" "74xx/74ls86.pdf" (at 41.91 124.46 0)
+      (effects (font (size 1.27 1.27)) hide)
+    )
+    (pin "3")
+    (pin "9")
+    (pin "7")
+    (pin "8")
+    (pin "14")
+    (pin "5")
+    (pin "13")
+    (pin "12")
+    (pin "11")
+    (pin "6")
+    (pin "4")
+    (pin "1")
+    (pin "10")
+    (pin "2")
+    (instances
+      (project "AppleII"
+        (path "/f1f08369-4db3-46f7-9b89-a5d3cfbed55a/00000000-0000-0000-0000-00006016cde0"
+          (reference "B2") (unit 5)
+        )
+      )
+    )
+  )
+  (symbol (lib_id "power:GND") (at 41.91 139.7 0) (unit 1)
+    (in_bom yes) (on_board yes) (dnp no)
+    (property "Reference" "#PWR013" (at 41.91 146.05 0)
+      (effects (font (size 1.27 1.27)) hide)
+    )
+    (property "Value" "GND" (at 45.212 141.224 0)
+      (effects (font (size 1.27 1.27)))
+    )
+    (property "Footprint" "" (at 41.91 139.7 0)
+      (effects (font (size 1.27 1.27)) hide)
+    )
+    (property "Datasheet" "" (at 41.91 139.7 0)
+      (effects (font (size 1.27 1.27)) hide)
+    )
+    (pin "1")
+    (instances
+      (project "AppleII"
+        (path "/f1f08369-4db3-46f7-9b89-a5d3cfbed55a/00000000-0000-0000-0000-00006016cde0"
+          (reference "#PWR013") (unit 1)
+        )
+      )

Commit message: Add files via upload
Other:
- note added: "Vertical Video Address"
Changed lines of the file:
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@@
     (effects (font (size 1.27 1.27) (thickness 0.254) bold) (justify left bottom))
+  )
+  (text "Vertical Video Address" (at 177.8 58.42 0)
+    (effects (font (size 1.27 1.27)) (justify left bottom))
   )
   (text "14.3 MHz Clock" (at 19.05 31.75 0)

Commit message: Add files via upload
Connections:
- net SOFT5: no longer B1.1 (~{CLR}), B2.4, C2.1 (~{MR})
- new net SOFT5a: B1.1 (~{CLR}), B2.4, C2.1 (~{MR})
Changed lines of the file:
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@@
     )
   )
-  (global_label "SOFT5" (shape input) (at 307.34 91.44 180)
+  (global_label "SOFT5a" (shape input) (at 307.34 91.44 180)
     (effects (font (size 1.27 1.27)) (justify right))
     (property "Intersheetrefs" "${INTERSHEET_REFS}" (at 307.34 91.44 0)
@@
     )
   )
-  (global_label "SOFT5" (shape input) (at 221.488 157.48 180)
+  (global_label "SOFT5a" (shape input) (at 221.488 157.48 180)
     (effects (font (size 1.27 1.27)) (justify right))
     (property "Intersheetrefs" "${INTERSHEET_REFS}" (at 221.488 157.48 0)
@@
     )
   )
-  (global_label "SOFT5" (shape input) (at 273.05 187.96 180)
+  (global_label "SOFT5a" (shape input) (at 273.05 187.96 180)
     (effects (font (size 1.27 1.27)) (justify right))
     (property "Intersheetrefs" "${INTERSHEET_REFS}" (at 273.05 187.96 0)

Commit message: Add files via upload
Parts:
- removed Q1, Q2: 2N4258, symbol Device:Q_PNP_BCE
- added unit 5 of A2
- added unit 5 of B13
- added Cap32, Cap33, Cap42, Cap43, Cap46, Cap48: 0.1uF, Apple-II:C_Disc_D5.0mm_W2.5mm_P5.00mm, symbol Device:C_Small
- added Q1, Q2: 2N4258, Package_TO_SOT_THT:TO-18-3, symbol Device:Q_PNP_EBC
- A2, B12, B13, B2, C11, D2: footprint Apple:DIP-14_W7.62mm -> Package_DIP:DIP-14_W7.62mm
- B1, C1, C2, D11, D12, D13, D14: footprint Apple:DIP-16_W7.62mm -> Package_DIP:DIP-16_W7.62mm
- B2: footprint (none) -> Package_DIP:DIP-14_W7.62mm
- Cap1: footprint (none) -> Apple-II:C_Disc_D5.0mm_W2.5mm_P5.00mm
- R1, R2, R3, R4: footprint Resistor_THT:R_Axial_DIN0207_L6.3mm_D2.5mm_P10.16mm_Horizontal -> Apple-II:R_Axial_DIN0207_L6.3mm_D2.5mm_P10.16mm_Horizontal
- Y1: footprint (none) -> Crystal:Crystal_HC18-U_Vertical
Connections:
- net SOFT5a is gone; now on net SOFT5: B1.1 (~{CLR}), B2.4, C2.1 (~{MR})
- net +12V: now also Cap48.1
- net +5V: now also A2.14 (VCC), B13.14 (VCC), Cap32.2, Cap33.2, Cap42.2, Cap43.2, Cap46.2, Q1.2 (B)
- net GND: now also A2.7 (GND), B13.7 (GND), Cap32.1, Cap33.1, Cap42.1, Cap43.1, Cap46.1, Cap48.2
- net at R4.2, Y1.2: now also Q2.2 (B)
- net at B2.10, R3.1: now also Q2.3 (C)
- net at R1.2: now also Q1.1 (E), Q2.1 (E)
- net at R2.1, Y1.1: now also Q1.3 (C)
Other:
- note removed: "Clock Generator"
- note removed: "Vertical Video Address"
- note removed: "Video Address Generator"
- moved on the sheet: A2A, B1, B12C, B13C, B2A, B2B, B2C, C1, C11D, C2, Cap1, D11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
