File: Connectors.kicad_sch (KiCad schematic)
At the start: 9 parts

Commit message: Add files via upload
Other:
- moved on the sheet: CP0, SLOT0, SLOT1, SLOT2, SLOT3, SLOT4, SLOT5, SLOT6, SLOT7

Commit message: Add files via upload
Connections:
- net ~{RESET} renamed ~{RST}

Commit message: Add files via upload
Connections:
- net P19: now reaches SLOT0.19 (Pin_19)
- net P19: now also SLOT1.19 (Pin_19), SLOT2.19 (Pin_19), SLOT3.19 (Pin_19), SLOT4.19 (Pin_19), SLOT5.19 (Pin_19), SLOT6.19 (Pin_19)
- net P35: now reaches SLOT0.35 (Pin_35)
- net P35: now also SLOT1.35 (Pin_35), SLOT2.35 (Pin_35), SLOT3.35 (Pin_35), SLOT4.35 (Pin_35), SLOT5.35 (Pin_35), SLOT6.35 (Pin_35)
- no-connect marks 21 -> 5

Commit message: Add files via upload
Changed lines of the file:
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@@
   )
   (no_connect (at 258.572 154.94))
-  (no_connect (at 269.24 148.082))
+  (no_connect (at 260.35 157.48))
   (no_connect (at 96.52 66.04))
   (no_connect (at 96.52 68.58))

Commit message: Add files via upload
Parts:
- CP0: footprint (none) -> Apple-II:POWER; DigiKey (none) -> A14226-ND
- SLOT0: footprint (none) -> Apple-II:Standard_Edge_Connector; DigiKey (none) -> A31718-ND
- SLOT1, SLOT2, SLOT3, SLOT4, SLOT5, SLOT6, SLOT7: footprint (none) -> Apple-II:Standard_Edge_Connector
Connections:
- net P19 is gone; now on net NC1: SLOT0.19 (Pin_19), SLOT1.19 (Pin_19), SLOT2.19 (Pin_19), SLOT3.19 (Pin_19), SLOT4.19 (Pin_19), SLOT5.19 (Pin_19), SLOT6.19 (Pin_19)
- net P35 is gone; now on net NC2: SLOT0.35 (Pin_35), SLOT1.35 (Pin_35), SLOT2.35 (Pin_35), SLOT3.35 (Pin_35), SLOT4.35 (Pin_35), SLOT5.35 (Pin_35), SLOT6.35 (Pin_35)
- net GND: now also SLOT4.26 (Pin_26)
- net NC1: now reaches SLOT7.19 (Pin_19)
- net NC2: now reaches SLOT7.35 (Pin_35)
- net ~{RST} renamed ~{RESET}
- no-connect marks 5 -> 4
