File: RAM.kicad_sch (KiCad schematic)
At the start: 26 parts

Commit message: Add files via upload
Connections:
- net LD0: no longer B8.10 (Q3)
- net LD1: no longer B8.12 (Q4)
- net LD2: no longer B8.5 (Q1)
- net LD3: no longer B8.7 (Q2)
- new net LD4: B8.10 (Q3)
- new net LD5: B8.12 (Q4)
- new net LD6: B8.5 (Q1)
- new net LD7: B8.7 (Q2)
Changed lines of the file:
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@@
     (effects (font (size 1.27 1.27)) (justify right bottom))
   )
-  (label "LD3" (at 148.59 181.61 180) (fields_autoplaced)
+  (label "LD7" (at 148.59 181.61 180) (fields_autoplaced)
     (effects (font (size 1.27 1.27)) (justify right bottom))
   )
@@
     (effects (font (size 1.27 1.27)) (justify right bottom))
   )
-  (label "LD0" (at 148.59 184.15 180) (fields_autoplaced)
+  (label "LD4" (at 148.59 184.15 180) (fields_autoplaced)
     (effects (font (size 1.27 1.27)) (justify right bottom))
   )
@@
     (effects (font (size 1.27 1.27)) (justify right bottom))
   )
-  (label "LD2" (at 148.59 179.07 180) (fields_autoplaced)
+  (label "LD6" (at 148.59 179.07 180) (fields_autoplaced)
     (effects (font (size 1.27 1.27)) (justify right bottom))
   )
@@
     (effects (font (size 1.27 1.27)) (justify left bottom))
   )
-  (label "LD1" (at 148.59 186.69 180) (fields_autoplaced)
-    (effects (font (size 1.27 1.27)) (justify right bottom))
-  )
+  (label "LD5" (at 148.59 186.69 180) (fields_autoplaced)
+    (effects (font (size 1.27 1.27)) (justify right bottom))
+  )

Commit message: Add files via upload
Other:
- note added: "Data Latch"
- moved on the sheet: B5, B8, C10, C3, C4, C5, C6, C7, C8, C9, D10, D3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

Commit message: Add files via upload
Other:
- note added: "B5-3, B5-2, B8-14, B8-15, B8-3, and B8-2 are all part of the video circuit."
- note added: "LD[0..7] = Latched Data bus feeding Video Generator sections"
- note removed: "LD0..7 = Latched Data bus feeding Video Generator sections"
- note removed: "Note: B5-3, B5-2, B8-14, B8-15, B8-3, and B8-2 are all part of the video circuit."
Changed lines of the file:
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@@
     (fill (type none))
   )
-  (text "LD0..7 = Latched Data bus\nfeeding Video Generator sections"
-    (at 186.182 214.122 0)
+  (text "LD[0..7] = Latched Data bus\nfeeding Video Generator sections"
+    (at 193.04 238.76 0)
     (effects (font (size 1.27 1.27)) (justify left bottom))
   )
@@
     (effects (font (size 1.27 1.27) bold) (justify left bottom))
   )
-  (text "Note:  B5-3, B5-2, B8-14, B8-15, \nB8-3, and B8-2 are all part of \nthe video circuit."
-    (at 138.43 265.43 0)
+  (text "B5-3, B5-2, B8-14, B8-15, \nB8-3, and B8-2 are all part of \nthe video circuit."
+    (at 193.04 251.46 0)
     (effects (font (size 1.27 1.27)) (justify left bottom))
   )
@@
     (effects (font (size 1.27 1.27)) (justify right bottom))
   )
-  (label "B5-3" (at 74.93 208.28 0) (fields_autoplaced)
-    (effects (font (size 1.27 1.27)) (justify left bottom))
-  )
   (label "RA3" (at 310.388 39.116 180) (fields_autoplaced)
     (effects (font (size 1.27 1.27)) (justify right bottom))
@@
     (effects (font (size 1.27 1.27)) (justify right bottom))
   )
-  (label "B11-5" (at 196.85 196.85 0) (fields_autoplaced)
-    (effects (font (size 1.27 1.27)) (justify left bottom))
-  )
   (label "RA4" (at 342.392 41.656 180) (fields_autoplaced)
     (effects (font (size 1.27 1.27)) (justify right bottom))
@@
     (effects (font (size 1.27 1.27)) (justify right bottom))
   )
-  (label "A8-6" (at 125.73 252.73 0) (fields_autoplaced)
-    (effects (font (size 1.27 1.27)) (justify left bottom))
-  )
   (label "LD5" (at 176.53 218.44 180) (fields_autoplaced)
     (effects (font (size 1.27 1.27)) (justify right bottom))
@@
     )
   )
+  (global_label "B11-5" (shape output) (at 204.47 196.85 0) (fields_autoplaced)
+    (effects (font (size 1.27 1.27)) (justify left))
+    (property "Intersheetrefs" "${INTERSHEET_REFS}" (at 213.2719 196.85 0)
+      (effects (font (size 1.27 1.27)) (justify left) hide)
+    )
+  )
   (global_label "RRW" (shape input) (at 277.114 104.902 180)
     (effects (font (size 1.27 1.27)) (justify right))
@@
     )
   )
+  (global_label "B5-3" (shape input) (at 72.39 208.28 180) (fields_autoplaced)
+    (effects (font (size 1.27 1.27)) (justify right))
+    (property "Intersheetrefs" "${INTERSHEET_REFS}" (at 64.7976 208.28 0)
+      (effects (font (size 1.27 1.27)) (justify right) hide)
+    )
+  )
   (global_label "RRW" (shape input) (at 179.578 57.658 180)
     (effects (font (size 1.27 1.27)) (justify right))
@@
     )
   )
+  (global_label "A8-6" (shape output) (at 133.35 252.73 0) (fields_autoplaced)
+    (effects (font (size 1.27 1.27)) (justify left))
+    (property "Intersheetrefs" "${INTERSHEET_REFS}" (at 140.761 252.73 0)
+      (effects (font (size 1.27 1.27)) (justify left) hide)
+    )
+  )

Commit message: Add files via upload
Connections:
- net A8-6: no longer names the net of B5.2 (Q0), B8.14 (D5)
Changed lines of the file:
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@@
   (junction (at 116.84 190.5) (diameter 0) (color 0 0 0 0)
   )
-  (junction (at 119.38 220.98) (diameter 0) (color 0 0 0 0)
-  )
   (junction (at 157.734 111.506) (diameter 0) (color 0 0 0 0)
   )
@@
     (stroke (width 0) (type default))
   )
-  (wire (pts (xy 119.38 220.98) (xy 119.38 252.73))
-    (stroke (width 0) (type default))
-  )
   (wire (pts (xy 255.27 63.754) (xy 287.274 63.754))
     (stroke (width 0) (type default))
@@
     (stroke (width 0) (type default))
   )
-  (wire (pts (xy 119.38 252.73) (xy 133.35 252.73))
-    (stroke (width 0) (type default))
-  )
   (wire (pts (xy 305.308 139.192) (xy 309.372 139.192))
     (stroke (width 0) (type default))
@@
     )
   )
-  (global_label "A8-6" (shape output) (at 133.35 252.73 0) (fields_autoplaced)
-    (effects (font (size 1.27 1.27)) (justify left))
-    (property "Intersheetrefs" "${INTERSHEET_REFS}" (at 140.761 252.73 0)
-      (effects (font (size 1.27 1.27)) (justify left) hide)
-    )
-  )

Commit message: Add files via upload
Connections:
- net SOFT5: no longer B5.1 (~{Mr})
- new net SOFT5a: B5.1 (~{Mr})
Changed lines of the file:
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@@
     )
   )
-  (global_label "SOFT5" (shape input) (at 80.01 231.14 180)
+  (global_label "SOFT5a" (shape input) (at 80.01 231.14 180)
     (effects (font (size 1.27 1.27)) (justify right))
     (property "Intersheetrefs" "${INTERSHEET_REFS}" (at 80.01 231.14 0)

Commit message: Add files via upload
Parts:
- added Cap20, Cap21, Cap22, Cap23, Cap24, Cap25, Cap26, Cap27, Cap28, Cap29, Cap3, Cap30, Cap31, Cap34, Cap35, Cap36, Cap37, Cap38, Cap39, Cap4, Cap40: 0.1uF, Apple-II:C_Disc_D5.0mm_W2.5mm_P5.00mm, symbol Device:C_Small
- B5, B8, C10, C3, C4, C5, C6, C7, C8, C9, D10, D3, D4, D5, D6, D7, D8, D9, E10, E3, E4, E5, E6, E7, E8, E9: footprint Apple:DIP-16_W7.62mm -> Package_DIP:DIP-16_W7.62mm
Connections:
- net SOFT5a is gone; now on net SOFT5: B5.1 (~{Mr})
- net +12V: now also Cap20.2, Cap22.2, Cap24.2, Cap25.2, Cap28.2, Cap29.2, Cap3.2, Cap31.2, Cap34.2, Cap37.2, Cap38.2, Cap40.2
- net +5V: now also Cap27.2, Cap35.2, Cap4.2
- net -5V: now also Cap21.2, Cap23.2, Cap26.2, Cap30.2, Cap36.2, Cap39.2
- net GND: now also Cap20.1, Cap21.1, Cap22.1, Cap23.1, Cap24.1, Cap25.1, Cap26.1, Cap27.1, Cap28.1, Cap29.1, Cap3.1, Cap30.1, Cap31.1, Cap34.1, Cap35.1, Cap36.1, Cap37.1, Cap38.1, Cap39.1, Cap4.1, Cap40.1
- net A8-6: now reaches B5.2 (Q0), B8.14 (D5)
Other:
- note added: "LD0..7 = Latched Data bus feeding Video Generator sections"
- note added: "Note: B5-3, B5-2, B8-14, B8-15, B8-3, and B8-2 are all part of the video circuit."
- note removed: "B5-3, B5-2, B8-14, B8-15, B8-3, and B8-2 are all part of the video circuit."
- note removed: "LD[0..7] = Latched Data bus feeding Video Generator sections"
