File: ROM.kicad_sch (KiCad schematic)
At the start: 8 parts

Commit message: Add files via upload
Parts:
- removed F12: 74LS138, Apple:DIP-16_W7.62mm, symbol 74xx:74LS138
- removed H1: 74LS08, Apple:DIP-14_W7.62mm, symbol 74xx:74LS08
Other:
- note removed: "C000-C7FF - to I/O Selects and Device Selects"
- note removed: "IO Strobe - goes to all Peripheral Connectors (slots) Goes low when accessing address range C800-C8FF"

Commit message: Add files via upload
Connections:
- net ROM_Select_D0 renamed ROM-SELECT-D0
- net ROM_Select_D8 renamed ROM-SELECT-D8
- net ROM_Select_E0 renamed ROM-SELECT-E0
- net ROM_Select_E8 renamed ROM-SELECT-E8
- net ROM_Select_F0 renamed ROM-SELECT-F0
- net ROM_Select_F8 renamed ROM-SELECT-F8

Commit message: Add files via upload
Parts:
- ROM-D0, ROM-D8, ROM-E0, ROM-E8, ROM-F0, ROM-F8: footprint Apple:DIP-24_W15.24mm -> Package_DIP:DIP-24_W15.24mm
Connections:
- net ROM-SELECT-D0 renamed ROM_SELECT_D0
- net ROM-SELECT-D8 renamed ROM_SELECT_D8
- net ROM-SELECT-E0 renamed ROM_SELECT_E0
- net ROM-SELECT-E8 renamed ROM_SELECT_E8
- net ROM-SELECT-F0 renamed ROM_SELECT_F0
- net ROM-SELECT-F8 renamed ROM_SELECT_F8
